File: _electronic/KiCad/esp32backup/e-tkt_esp32.kicad_sch (KiCad schematic)
At the start: 64 parts, among them J2 USB4120-03-C_REVA, Q1 SS8050-G, Q2 SS8050-G, U2 AZ1117I-3.3, U6 ESP32-S3-WROOM-1-N8R2

Commit message: pcb draft with esp32-s3
Parts:
- removed C1: 0.1uF/50v(10%), Capacitor_SMD:C_0603_1608Metric_Pad1.08x0.95mm_HandSolder, symbol Device:C
- removed D2, D_RX1, D_TX1: LED, LED_SMD:LED_0805_2012Metric, symbol Device:LED
- removed R1: 10K(5%), Resistor_SMD:R_0603_1608Metric, symbol Device:R
- removed R2, R3: 470R, Resistor_SMD:R_0603_1608Metric_Pad0.98x0.95mm_HandSolder, symbol Device:R
- removed R4: 10K, Resistor_SMD:R_0603_1608Metric_Pad0.98x0.95mm_HandSolder, symbol Device:R
- removed S_BOOT1, S_RESET1, S_WIFIRESET1: TS06-667-25-BK-100-G-SMT-TR, SnapEDA Library:SW_TS06-667-25-BK-100-G-SMT-TR, symbol TS06-667-25-BK-100-G-SMT-TR:TS06-667-25-BK-100-G-SMT-TR
- added C16: 100nF, Capacitor_SMD:C_0805_2012Metric, symbol Device:C
- added C5: 0.1uF/50v(10%), Capacitor_SMD:C_0805_2012Metric, symbol Device:C
- added D4: LED, LED_SMD:LED_0805_2012Metric, symbol Device:LED
- added R9: 10K(5%), Resistor_SMD:R_0805_2012Metric, symbol Device:R
- added S_ENABLE1, S_REBOOT1, S_WIFI_RESET1: PTS645SM43SMTR92_LFS, digikey-footprints:Switch_Tactile_SMD_6x6mm_PTS645, symbol dk_Tactile-Switches:PTS645SM43SMTR92_LFS
- added U1: ESP32-WROOM-32D, RF_Module:ESP32-WROOM-32, symbol RF_Module:ESP32-WROOM-32D
- added U4: FT231XS, Package_SO:SSOP-20_3.9x8.7mm_P0.635mm, symbol Interface_USB:FT231XS
- A_DRIVER1: footprint SnapEDA Library:Pololu_Breakout-16_15.2x20.3mm -> Module:Pololu_Breakout-16_15.2x20.3mm
- C10, C11, C13, C14, C15, C17, C3, C4, C6, C7: footprint Capacitor_SMD:C_0603_1608Metric_Pad1.08x0.95mm_HandSolder -> Capacitor_SMD:C_0805_2012Metric
- C12, C18, C8, C9: footprint Capacitor_Tantalum_SMD:CP_EIA-1608-10_AVX-L_Pad1.25x1.05mm_HandSolder -> Capacitor_Tantalum_SMD:CP_EIA-1608-10_AVX-L
- D5, D6, D7, D8: footprint LED_SMD:LED_0603_1608Metric_Pad1.05x0.95mm_HandSolder -> LED_SMD:LED_0805_2012Metric
- F2: footprint Fuse:Fuse_1210_3225Metric_Pad1.42x2.65mm_HandSolder -> Fuse:Fuse_1210_3225Metric
- FB1: footprint Inductor_SMD:L_0603_1608Metric_Pad1.05x0.95mm_HandSolder -> Inductor_SMD:L_0805_2012Metric
- J_masterpower1: footprint SnapEDA Library:BarrelJack_GCT_DCJ200-10-A_Horizontal -> Connector_BarrelJack:BarrelJack_GCT_DCJ200-10-A_Horizontal
- Q1, Q2: footprint Package_TO_SOT_SMD:SOT-23 -> digikey-footprints:SOT-23-3
- R10, R11, R12, R13, R15, R16, R17, R18, R7, R8: footprint Resistor_SMD:R_0603_1608Metric -> Resistor_SMD:R_0805_2012Metric
- R19, R20, R21, R22: footprint Resistor_SMD:R_0603_1608Metric_Pad0.98x0.95mm_HandSolder -> Resistor_SMD:R_0805_2012Metric
- U2: footprint Package_TO_SOT_SMD:SOT-223 -> digikey-footprints:SOT-223
- U6: value ESP32-S3-WROOM-1-N8R2 -> ESP32-S3-WROOM-1-N16R2
Connections:
- net +12V: now also C10.1, S_power1.5, U2.3 (IN); no longer S_power1.1
- net +3.3V: now also D4.2 (A), R9.1, S_WIFI_RESET1.1, S_WIFI_RESET1.2, U1.2 (VDD); no longer U2.4 (VOUT), U6.2 (3V3)
- net DTR: now also U4.1 (~{DTR})
- net EN: now also C5.1, R9.2, S_ENABLE1.3, S_ENABLE1.4, U1.3 (EN); no longer U6.3 (EN)
- net GNDREF: now also C16.1, C5.2, S_ENABLE1.1, S_ENABLE1.2, S_REBOOT1.1, S_REBOOT1.2, U1.1 (GND), U1.15 (GND), U1.38 (GND), U1.39 (GND), U4.16 (GND), U4.6 (GND); no longer J_masterpower1.2, J_masterpower1.3, S_power1.2, S_power1.6, U6.1 (GND), U6.40 (GND), U6.41_1 (GND), U6.41_2 (GND), U6.41_3 (GND), U6.41_4 (GND), U6.41_5 (GND), U6.41_6 (GND), U6.41_7 (GND), U6.41_8 (GND), U6.41_9 (GND)
- net IO0: now also S_REBOOT1.3, S_REBOOT1.4, U1.25 (IO0); no longer U6.27 (IO0)
- net IO1: now also U1.35 (TXD0/IO1), U4.4 (RXD); no longer U6.39 (IO1)
- net IO12: now also U1.14 (IO12); no longer U6.20 (IO12), U_DRIVER1.3 (I3)
- net IO13: now also S_WIFI_RESET1.3, S_WIFI_RESET1.4, U1.16 (IO13); no longer U6.21 (IO13), U_DRIVER1.2 (I2)
- net IO14: now also Q_SERVO1.2 (S), R13.1, U1.13 (IO14); no longer U6.22 (IO14), U_DRIVER1.1 (I1)
- net IO15: now also U_DRIVER1.1 (I1), U1.23 (IO15); no longer U6.8 (IO15)
- net IO16: now also U_DRIVER1.4 (I4), U1.27 (IO16); no longer U6.9 (IO16)
- net IO17: now also J_LED_CAROUSEL1.2 (Pin_2), U1.28 (IO17); no longer U6.10 (IO17)
- net IO18: now also U1.30 (IO18); no longer U6.11 (IO18)
- net IO19: now also U1.31 (IO19); no longer R19.2, U6.13 (IO19)
- net IO2: now also U_DRIVER1.3 (I3), U1.24 (IO2); no longer U6.38 (IO2)
- net IO21: now also J_OLED1.4 (Pin_4), U1.33 (IO21); no longer U6.23 (IO21)
- net IO3: now also U1.34 (RXD0/IO3), U4.20 (TXD); no longer U6.15 (IO3)
- net IO35: now also U1.7 (IO35); no longer A_DRIVER1.9 (~{ENABLE}), U6.28 (IO35)
- net IO4: now also U_DRIVER1.2 (I2), U1.26 (IO4); no longer U6.4 (IO4)
- net IO5: now also J_LED_FINISH1.2 (Pin_2), U1.29 (IO5); no longer U6.5 (IO5)
- net RTS: now also U4.2 (~{RTS})
- net at C11.1: now also D4.1 (K)
- net at J_masterpower1.1: now also S_power1.1; no longer S_power1.5
- net +5V: no longer names the net of C17.2, C18.1, F2.2
- net +5V: now also U4.15 (VCC); no longer S_power1.7
- removed net IO10: Q_SERVO1.2 (S), R13.1, U6.18 (IO10)
- net IO11: no longer names the net of U6.19 (IO11)
- net IO11: no longer U_DRIVER1.4 (I4)
- net IO20: no longer names the net of U6.14 (IO20)
- net IO20: no longer R20.1
- net IO36: no longer names the net of U6.29 (IO36)
- net IO36: no longer A_DRIVER1.15 (STEP)
- net IO37: no longer names the net of U6.30 (IO37)
- net IO37: no longer J_LED_CAROUSEL1.2 (Pin_2)
- net IO38: no longer names the net of U6.31 (IO38)
- net IO38: no longer J_LED_FINISH1.2 (Pin_2)
- net IO39: no longer names the net of U6.32 (IO39)
- net IO40: no longer names the net of U6.33 (IO40)
- net IO41: no longer names the net of U6.34 (IO41)
- net IO42: no longer names the net of U6.35 (IO42)
- net IO45: no longer names the net of U6.26 (IO45)
- net IO45: no longer A_DRIVER1.16 (DIR)
- net IO46: no longer names the net of U6.16 (IO46)
- net IO47: no longer names the net of U6.24 (IO47)
- net IO47: no longer J_OLED1.4 (Pin_4)
- net IO48: no longer names the net of U6.25 (IO48)
- net IO48: no longer J_OLED1.3 (Pin_3)
- net IO6: no longer names the net of U6.6 (IO6)
- net IO7: no longer names the net of U6.7 (IO7)
- net IO8: no longer names the net of U6.12 (IO8)
- net IO9 renamed IO34
- net IO34: now also U1.6 (IO34); no longer U6.17 (IO9)
- removed net VIN: C10.1, S_power1.3, U2.3 (IN)
- new net: U6.1 (GND), U6.40 (GND), U6.41_1 (GND), U6.41_2 (GND), U6.41_3 (GND), U6.41_4 (GND), U6.41_5 (GND), U6.41_6 (GND), U6.41_7 (GND), U6.41_8 (GND), U6.41_9 (GND)
- new net: J_masterpower1.3, S_power1.2, S_power1.3
- new net: R19.2, U4.12 (USBDM)
- new net: R20.1, U4.11 (USBDP)
- new net: C16.2, U4.13 (3V3OUT), U4.14 (~{RESET}), U4.3 (VCCIO)
- new net IO22: J_OLED1.3 (Pin_3), U1.36 (IO22)
- new net IO23: U1.37 (IO23)
- new net IO25: A_DRIVER1.9 (~{ENABLE}), U1.10 (IO25)
- new net IO26: U1.11 (IO26)
- new net IO27: U1.12 (IO27)
- new net IO32: A_DRIVER1.15 (STEP), U1.8 (IO32)
- new net IO33: A_DRIVER1.16 (DIR), U1.9 (IO33)
- no-connect marks 13 -> 22
Other:
- note added: "12V POWER"
- note added: "ESP32"
- note added: "REBOOT / ENABLE"
- note removed: "5v on barrel pin 3?"
- note removed: "9-12V EXTERNAL POWER"
- note removed: "DIODE?"
- note removed: "ESP32-S3"
- note removed: "LED voltage resistors values (5-12v?)"
- note removed: "RESET / BOOT"
- note removed: "reatribute pins (from ESP32 to ESP32-S3)"
- moved on the sheet: A_DRIVER1, C10, C11, C12, C13, C14, C15, C17, C18, C3, C4, C6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
