File: _electronic/KiCad/e-tkt.kicad_pcb (KiCad board)
At the start: 2 copper layers, 99.6 x 72.7 mm, 90 parts, among them J1 USB4105-GF-A, Q1 SS8050-G, Q2 SS8050-G, U1 USB6B1, U2 AZ1117I-3.3, U3 FT231XS, U4 ESP32-WROOM-32

Commit message: board silhouette and ftdi
Parts:
- removed TP_IO15, TP_IO18, TP_IO5, TP_IO6, TP_IO7, TP_IO8: TestPoint, TestPoint:TestPoint_Pad_D1.0mm
- added C13: 47pF, Capacitor_SMD:C_0603_1608Metric_Pad1.08x0.95mm_HandSolder, F.Cu at (148.8, -195.6)
- added C15: 0.1uF, Capacitor_SMD:C_0603_1608Metric_Pad1.08x0.95mm_HandSolder, F.Cu at (145.3, -187.4)
- added C16: 0.1uF, Capacitor_SMD:C_0603_1608Metric_Pad1.08x0.95mm_HandSolder, F.Cu at (152.5, -197.6)
- added C5: 47pF, Capacitor_SMD:C_0603_1608Metric_Pad1.08x0.95mm_HandSolder, F.Cu at (148.8, -191.0)
- added D_RX1: LED, LED_SMD:LED_0603_1608Metric_Pad1.05x0.95mm_HandSolder, F.Cu at (160.5, -192.0)
- added D_TX1: LED, LED_SMD:LED_0603_1608Metric_Pad1.05x0.95mm_HandSolder, F.Cu at (160.5, -194.1)
- added JP4: SolderJumper_2_Bridged, Jumper:SolderJumper-2_P1.3mm_Bridged2Bar_Pad1.0x1.5mm, B.Cu at (153.9, -202.2)
- added JP5: SolderJumper_2_Bridged, Jumper:SolderJumper-2_P1.3mm_Bridged2Bar_Pad1.0x1.5mm, B.Cu at (156.5, -202.2)
- added JP6: SolderJumper_2_Bridged, Jumper:SolderJumper-2_P1.3mm_Bridged2Bar_Pad1.0x1.5mm, B.Cu at (178.3, -191.0)
- added JP7: SolderJumper_2_Bridged, Jumper:SolderJumper-2_P1.3mm_Bridged2Bar_Pad1.0x1.5mm, B.Cu at (178.3, -188.5)
- added R14: 27R, Resistor_SMD:R_0603_1608Metric_Pad0.98x0.95mm_HandSolder, F.Cu at (148.8, -192.5)
- added R19: 27R, Resistor_SMD:R_0603_1608Metric_Pad0.98x0.95mm_HandSolder, F.Cu at (148.8, -194.1)
- C12, C9: value 10uF -> 10uF/25v; footprint Capacitor_Tantalum_SMD:CP_EIA-3216-10_Kemet-I_Pad1.58x1.35mm_HandSolder -> Capacitor_SMD:C_0603_1608Metric_Pad1.08x0.95mm_HandSolder
- moved J_SERVO1 6.67 mm to (187.2, -164.1), turned to 90 degrees
- moved J_USBPOWER1 4.79 mm to (141.2, -182.4), turned to 180 degrees
- moved D9 4.77 mm to (212.4, -193.5), turned to 0 degrees
- moved C12 4.19 mm to (151.3, -178.9), turned to -90 degrees
- moved H2 3.56 mm to (221.0, -224.0)
- moved H3 3.56 mm to (221.0, -158.5)
- moved H5 3.56 mm to (221.0, -191.5)
- moved H1 3.56 mm to (135.6, -224.0)
- moved H4 3.56 mm to (135.6, -158.5)
- moved D5 3.43 mm to (164.2, -171.2)
- moved D6 3.43 mm to (160.1, -171.2)
- moved D7 3.43 mm to (156.1, -171.2)
- moved D8 3.43 mm to (152.1, -171.2)
- moved J_28byj-48-12v_1 3.43 mm to (163.7, -164.1)
- moved J_masterpower1 3.43 mm to (146.2, -171.2)
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Connections:
- net /DTR renamed DTR
- net /RTS renamed RTS
- net IO13 renamed IO13 WIFI RST
- net IO14 renamed IO14 SERVO
- net IO15 renamed IO15 ULN 1
- net IO16 renamed IO16 ULN 4
- net IO17 renamed IO17 LED PRESS
- net IO2 renamed IO2 ULN 3
- net IO21 renamed IO21 OLED SDA
- net IO22 renamed IO22 OLED SCL
- net IO25 renamed IO25 NEMA ENA
- net IO32 renamed IO32 NEMA STEP
- net IO33 renamed IO33 NEMA DIR
- net IO34 renamed IO34 HALL
- net IO4 renamed IO4 ULN 2
- net IO5 renamed IO5 LED END
- C12 pad 1: +12V -> GNDREF
- C12 pad 2: GNDREF -> +12V
- C9 pad 1: +3.3V -> GNDREF
- C9 pad 2: GNDREF -> +3.3V
- J_USBPOWER1 pad 1: +12V -> +5V
- J_USBPOWER1 pad 2: +5V -> +12V
- TP_RX1 pad 1: TXD0 IO1 -> IO1 TXD
- TP_TX1 pad 1: RXD0 IO3 -> IO3 RXD
- U3 pad 1: unconnected-(U3-Pad1) -> Net-(U3-Pad1)
- U3 pad 10: unconnected-(U3-Pad10) -> Net-(U3-Pad10)
- U3 pad 11: D+ -> Net-(R19-Pad1)
- U3 pad 12: D- -> Net-(R14-Pad1)
- U3 pad 13: unconnected-(U3-Pad13) -> +3.3V
- U3 pad 14: unconnected-(U3-Pad14) -> +3.3V
- U3 pad 15: unconnected-(U3-Pad15) -> +5V
- U3 pad 16: unconnected-(U3-Pad16) -> GNDREF
- U3 pad 17: unconnected-(U3-Pad17) -> Net-(U3-Pad17)
- U3 pad 2: unconnected-(U3-Pad2) -> Net-(U3-Pad2)
- U3 pad 20: RXD0 IO3 -> Net-(U3-Pad20)
- U3 pad 3: unconnected-(U3-Pad3) -> +3.3V
- U3 pad 4: TXD0 IO1 -> Net-(U3-Pad4)
- U4 pad 11: IO26 -> unconnected-(U4-Pad11)
- U4 pad 12: IO27 -> unconnected-(U4-Pad12)
- U4 pad 14: IO12 -> unconnected-(U4-Pad14)
- U4 pad 30: IO18 -> unconnected-(U4-Pad30)
- U4 pad 31: IO19 -> unconnected-(U4-Pad31)
- U4 pad 34: RXD0 IO3 -> IO3 RXD
- U4 pad 35: TXD0 IO1 -> IO1 TXD
- U4 pad 37: IO23 -> unconnected-(U4-Pad37)
- U4 pad 7: IO35 -> unconnected-(U4-Pad7)
Routing:
- net RXD0 IO3: track 65.5 -> 0.00 mm, vias 3 -> 0
- net TXD0 IO1: track 64.3 -> 0.00 mm, vias 3 -> 0
- net +12V: track 185.0 -> 243.5 mm, vias 7 -> 11
- net IO3 RXD: track 0.00 -> 51.7 mm, vias 0 -> 4
- net IO1 TXD: track 0.00 -> 50.6 mm, vias 0 -> 2
- net +3.3V: track 256.0 -> 292.5 mm, vias 8 -> 11
- net DTR: track 1.92 -> 34.4 mm, vias 0 -> 3
- net +6V: track 119.9 -> 150.3 mm
- net GNDREF: track 29.7 -> 57.2 mm, vias 253 -> 252
- net RTS: track 1.92 -> 28.4 mm, vias 0 -> 1
- net Net-(U3-Pad2): track 0.00 -> 22.2 mm, vias 0 -> 1
- net Net-(U3-Pad1): track 0.00 -> 21.0 mm, vias 0 -> 1
- net SERVO: track 2.39 -> 21.2 mm
- net Net-(U3-Pad20): track 0.00 -> 16.6 mm, vias 0 -> 1
- net Net-(U3-Pad4): track 0.00 -> 13.2 mm, vias 0 -> 1
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Other:
- board size 99.6 x 72.7 mm -> 96 x 72.7 mm
- board text added: "12v 3A"
- board text added: "Andrei Speridião 2022/07/09 v0.9"
- board text added: "CUT"
- board text added: "EXTERNAL FLASHING"
- board text added: "ON"
- board text added: "USB"
- board text removed: "05"
- board text removed: "06"
- board text removed: "07"
- board text removed: "08"
- board text removed: "15"
- board text removed: "18"
- board text removed: "2022/07/07"
- board text removed: "GPIOs"
- board text removed: "v0.9"
