File: _electronic/KiCad/e-tkt.kicad_sch (KiCad schematic)
At the start: 96 parts, among them J1 USB4105-GF-A, Q1 SS8050-G, Q2 SS8050-G, U1 USB6B1, U2 AZ1117I-3.3, U3 FT231XS, U4 ESP32-WROOM-32

Commit message: led resistors, better pcb layout, omron tact
Parts:
- removed S_BOOT1, S_RESET1, S_WIFIRESET1: TS06-667-25-BK-100-G-SMT-TR, SnapEDA Library:SW_TS06-667-25-BK-100-G-SMT-TR, symbol TS06-667-25-BK-100-G-SMT-TR:TS06-667-25-BK-100-G-SMT-TR
- added R22, R23, R24, R25, R26, R27: 47R, Resistor_SMD:R_0603_1608Metric, symbol Device:R
- added SW1, SW2, SW3: B3FS-1000, b3fs:B3FS-1000, symbol 2022-07-12_23-59-33:B3FS-1000
- R20, R21: value 0R -> 47R
Connections:
- net EN: now also SW2.3, SW2.4
- net GNDREF: now also D1.1 (K), D4.1 (K), SW1.1, SW1.2, SW2.1, SW2.2, SW3.1, SW3.2
- net IO0 RESET: now also SW1.3, SW1.4
- net IO13 WIFI RST: now also SW3.3, SW3.4
- net IO14 SERVO: now also R25.1; no longer D10.2 (A)
- net IO25 NEMA ENA: now also A_DRIVER1.9 (~{ENABLE}), R26.1; no longer D4.2 (A)
- net IO32 NEMA STEP: now also A_DRIVER1.15 (STEP), R27.2; no longer D1.2 (A)
- net IO34 HALL: now also R24.1; no longer D9.2 (A)
- net at D_RX1.1 (K): now also R22.1; no longer U3.17 (CBUS1)
- net at D_TX1.1 (K): now also R23.1; no longer U3.10 (CBUS2)
- new net: R23.2, U3.10 (CBUS2)
- new net: R22.2, U3.17 (CBUS1)
- new net: D1.2 (A), R27.1
- new net: D4.2 (A), R26.2
- new net: D9.2 (A), R24.2
- new net: D10.2 (A), R25.2
- no-connect marks 32 -> 29
Other:
- moved on the sheet: A_DRIVER1, C1, C10, C11, C12, C3, C8, C9, D1, D10, D11, D4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

Commit message: rev1 schematics export
Parts:
- renumbered U_6v2 to U5, U_DRIVER1 to U6
Connections:
- net D1+ renamed USBD1+
- net D1- renamed USBD1-
Other:
- note added: "BOOT & RESET"
- note added: "PADS / TESTING"
- note added: "Question: how to keep the usb plugged while having external 12v supplied, without problems? I.E. 12v going back to 5v, floating ground, etc..."
- note removed: "BOOT / RESET"
- note removed: "PADS"
- moved on the sheet: A_DRIVER1, C1, C10, C11, C12, C13, C14, C15, C16, C17, C2, C3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

Commit message: ftdi revision, removed usb vcc jumper
Parts:
- removed D2: BAT760,115, Diode_SMD:D_SOD-323, symbol Diode:BAT41
- removed J_USBPOWER1: Conn_01x02_Male, Connector_PinHeader_2.54mm:PinHeader_1x02_P2.54mm_Vertical, symbol Connector:Conn_01x02_Male
- added F1: 6V 40A 750mA, Fuse:Fuse_0805_2012Metric_Pad1.15x1.40mm_HandSolder, symbol Device:Polyfuse
- added FB1: 6V 750mA, Inductor_SMD:L_0805_2012Metric_Pad1.05x1.20mm_HandSolder, symbol Device:FerriteBead
Connections:
- net +12V: no longer C10.1, U2.3 (IN)
- net +6V: now also C10.1, U2.3 (IN)
- net at J1.A4_B9 (VBUS), J1.B4_A9 (VBUS), U1.1 (VBUS)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: now also F1.1
- net +5V renamed VBUS
- net VBUS: now also FB1.2
- new net: F1.2, FB1.1
Other:
- note added: "hall: voltage divider"
- note added: "servo, mosfet"
- note removed: "Question: how to keep the usb plugged while having external 12v supplied, without problems? I.E. 12v going back to 5v, floating ground, etc..."
- moved on the sheet: A_DRIVER1, C10, C11, C13, C14, C15, C17, C2, C5, C8, C9, D1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

Commit message: bucket 6v and latch power
Parts:
- removed C17: 0.1uF, Capacitor_SMD:C_0603_1608Metric_Pad1.08x0.95mm_HandSolder, symbol Device:C
- removed U5: L7806, Package_TO_SOT_SMD:TO-263-2, symbol Regulator_Linear:L7806
- added 11uH/15.8mOhm1: SRP6060FA-100M, SRP6060FA:SRP6060FA-4R7M, symbol Device:L
- added C18: 22uF, Capacitor_SMD:C_0603_1608Metric_Pad1.08x0.95mm_HandSolder, symbol Device:C
- added C_BST1: 100nF 64mOhm, Capacitor_SMD:C_0603_1608Metric_Pad1.08x0.95mm_HandSolder, symbol Device:C
- added C_FF1: 82pF/0Ohm, Capacitor_SMD:C_0603_1608Metric_Pad1.08x0.95mm_HandSolder, symbol Device:C
- added C_IN1, C_IN2, C_IN3: 10uF/5mOhm, Capacitor_SMD:C_1210_3225Metric_Pad1.33x2.70mm_HandSolder, symbol Device:C
- added C_OUT1, C_OUT2, C_OUT3, C_OUT4, C_OUT5: 22uF/1mOhm, Capacitor_SMD:C_1210_3225Metric_Pad1.33x2.70mm_HandSolder, symbol Device:C
- added D2: LED, LED_SMD:LED_0603_1608Metric_Pad1.05x0.95mm_HandSolder, symbol Device:LED
- added Q3: AO3401A, Package_TO_SOT_SMD:SOT-23, symbol dk_Transistors-FETs-MOSFETs-Single:AO3401A
- added Q4, Q5: 2SC4213, Package_TO_SOT_SMD:SOT-23, symbol Transistor_BJT:2SC4213
- added R28: 430R, Resistor_SMD:R_0603_1608Metric_Pad0.98x0.95mm_HandSolder, symbol Device:R
- added R29, R30, R32, R_FBT1: 100K, Resistor_SMD:R_0603_1608Metric_Pad0.98x0.95mm_HandSolder, symbol Device:R
- added R31: 1M, Resistor_SMD:R_0603_1608Metric_Pad0.98x0.95mm_HandSolder, symbol Device:R
- added R_FFB1: 11K, Resistor_SMD:R_0603_1608Metric_Pad0.98x0.95mm_HandSolder, symbol Device:R
- added SW4: B3FS-1000, b3fs:B3FS-1000, symbol 2022-07-12_23-59-33:B3FS-1000
- added U5: TPS54302, Package_TO_SOT_SMD:SOT-23-6, symbol Regulator_Switching:TPS54302
- C14: value 0.33uF -> 22uF/1mOhm; footprint Capacitor_SMD:C_0603_1608Metric_Pad1.08x0.95mm_HandSolder -> Capacitor_SMD:C_1210_3225Metric_Pad1.33x2.70mm_HandSolder; Id (none) -> C1608JB1A226M080AC
- Q_HALL1, Q_SERVO1: footprint Package_TO_SOT_SMD:SOT-323_SC-70 -> Package_TO_SOT_SMD:SOT-23
- R2: footprint Resistor_SMD:R_0603_1608Metric -> Resistor_SMD:R_0603_1608Metric_Pad0.98x0.95mm_HandSolder
Connections:
- net +12V: now also C_IN1.1, C_IN2.1, C_IN3.1, Q3.3 (D), R30.2, R31.2, U5.3 (VIN); no longer C14.1, J_masterpower1.1
- net +6V: now also C14.1, 11uH/15.8mOhm1.2, C_FF1.1, C_OUT1.1, C_OUT2.1, C_OUT3.1, C_OUT4.1, C_OUT5.1, R_FBT1.2
- net GNDREF: now also J_LED_END1.1 (Pin_1), J_LED_PRESS1.1 (Pin_1), C18.2, C_IN1.2, C_IN2.2, C_IN3.2, C_OUT1.2, C_OUT2.2, C_OUT3.2, C_OUT4.2, C_OUT5.2, D2.1 (K), Q4.2 (E), Q5.2 (E), R_FFB1.1, U5.1 (GND); no longer R20.2, R21.2
- net IO17 LED PRESS: now also R20.1; no longer J_LED_PRESS1.2 (Pin_2)
- net IO5 LED END: now also R21.1; no longer J_LED_END1.2 (Pin_2)
- new net: Q3.1 (G), Q4.3 (C), R29.1
- new net: C_BST1.1, U5.6 (BOOT)
- new net: 11uH/15.8mOhm1.1, C_BST1.2, U5.2 (SW)
- new net: C18.1, Q5.1 (B), R31.1
- new net: Q5.3 (C), R32.1, SW4.3, SW4.4
- new net: C_FF1.2, R_FBT1.1, R_FFB1.2, U5.4 (FB)
- new net: D2.2 (A), R28.2
- new net: J_LED_END1.2 (Pin_2), R21.2
- new net: Q4.1 (B), R30.1, SW4.1, SW4.2
- new net: J_LED_PRESS1.2 (Pin_2), R20.2
- new net POWER IN: J_masterpower1.1, Q3.2 (S), R28.1, R29.2, R32.2
- no-connect marks 29 -> 30
Other:
- note added: "6V POWER: BUCK"
- note added: "LATCH POWER"
- moved on the sheet: D11, J_LED_END1, J_OLED1, J_SERVO1, J_masterpower1, R2, R20, R21

Commit message: added vias, revised parts, fixed schematic
Parts:
- A_NEMA1: renamed from A_DRIVER1; value Pololu_Breakout_A4988 -> 8+8 pin; # (none) -> M20-7820842 (2 units); Group (none) -> NEMA; Mouser (none) -> OK
- C_ENA1: renamed from C4; value 0.1uF/50v(10%) -> 0.1uF 10V; # (none) -> CGA3E2X7R1H104K080AA; Group (none) -> Enable; Id CGA3E2X7R1H104K080AA -> (none); Mouser (none) -> OK
- C_MCU1: renamed from C7; value 0.1uF/50v(10%) -> 0.1uF 10V; # (none) -> CGA3E2X7R1H104K080AA; Group (none) -> MCU; Id CGA3E2X7R1H104K080AA -> (none); Mouser (none) -> OK
- C_MCU2: renamed from C6; value 22uF/10V(20%) -> 22uF 12V 1mOhm; # (none) -> CL10A226MO7JZNC; Group (none) -> MCU; Id C1608JB1A226M080AC -> (none); Mouser (none) -> OK; Obs (none) -> wes
- C_NEMA1: renamed from C8; value 100uF -> 100uF 25V; # (none) -> EMVE250ADA101MF80G; Group (none) -> NEMA; Id 16TZV100M6.3X6.1 -> (none); Mouser (none) -> OK
- C_NEMA2: renamed from C9; value 10uF/25v -> 10uF 12V 5mOhm; # (none) -> C1608X5R1E106M080AC; Group (none) -> NEMA; Id C1608X5R1E106M080AC -> (none); Mouser (none) -> OK; Obs (none) -> wes
- C_POW1: renamed from C10; value 10uF/10V(20%) -> 10uF 12V 5mOhm; # (none) -> C1608X5R1E106M080AC; Group (none) -> 3V3 power; Mouser (none) -> OK; Obs (none) -> wes
- C_POW2: renamed from C11; value 22uF/10V(20%) -> 22uF 12V 1mOhm; # (none) -> CL10A226MO7JZNC; Group (none) -> 3V3 power; Id C1608JB1A226M080AC -> (none); Mouser (none) -> OK; Obs (none) -> wes
- C_POW3: renamed from C18; value 22uF -> 22uF 12V 1mOhm; # (none) -> CL10A226MO7JZNC; Group (none) -> Latch power; Id C1608JB1A226M080AC -> (none); Mouser (none) -> OK; Obs (none) -> wes
- C_POW_6V_FF1: renamed from C_FF1; value 82pF/0Ohm -> 82pF 6V 0Ohm; # (none) -> VJ0603A820JXBAC; Group (none) -> 6V power; Id C1608JB1A226M080AC -> (none); Mouser (none) -> OK; Obs (none) -> wes
- C_POW_BST1: renamed from C_BST1; value 100nF 64mOhm -> 100nF 6V 64mOhm; # (none) -> C1608X7R1H104K080AA; Group (none) -> 6V power; Id C1608JB1A226M080AC -> (none); Mouser (none) -> OK
- C_POW_IN1: renamed from C_IN1; value 10uF/5mOhm -> 10uF 12V 5mOhm; # (none) -> C1608X5R1E106M080AC; Group (none) -> 6V power; Id C1608JB1A226M080AC -> (none); Mouser (none) -> OK; Obs (none) -> wes
- C_POW_IN2: renamed from C_IN2; value 10uF/5mOhm -> 10uF 12V 5mOhm; # (none) -> C1608X5R1E106M080AC; Group (none) -> 6V power; Id C1608JB1A226M080AC -> (none); Mouser (none) -> OK; Obs (none) -> wes
- C_POW_IN3: renamed from C_IN3; value 10uF/5mOhm -> 10uF 12V 5mOhm; # (none) -> C1608X5R1E106M080AC; Group (none) -> 6V power; Id C1608JB1A226M080AC -> (none); Mouser (none) -> OK; Obs (none) -> wes
- C_POW_OUT1: renamed from C_OUT1; value 22uF/1mOhm -> 22uF 12V 1mOhm; # (none) -> C3225X7R1E226M250AB; Group (none) -> 6V power; Id C1608JB1A226M080AC -> (none); Mouser (none) -> OK; Obs (none) -> wes
- C_POW_OUT2: renamed from C_OUT2; value 22uF/1mOhm -> 22uF 12V 1mOhm; # (none) -> C3225X7R1E226M250AB; Group (none) -> 6V power; Id C1608JB1A226M080AC -> (none); Mouser (none) -> OK; Obs (none) -> wes
- C_POW_OUT3: renamed from C_OUT3; value 22uF/1mOhm -> 22uF 12V 1mOhm; # (none) -> C3225X7R1E226M250AB; Group (none) -> 6V power; Id C1608JB1A226M080AC -> (none); Mouser (none) -> OK; Obs (none) -> wes
- C_POW_OUT4: renamed from C_OUT4; value 22uF/1mOhm -> 22uF 12V 1mOhm; # (none) -> C3225X7R1E226M250AB; Group (none) -> 6V power; Id C1608JB1A226M080AC -> (none); Mouser (none) -> OK; Obs (none) -> wes
- C_POW_OUT5: renamed from C_OUT5; value 22uF/1mOhm -> 22uF 12V 1mOhm; # (none) -> C3225X7R1E226M250AB; Group (none) -> 6V power; Id C1608JB1A226M080AC -> (none); Mouser (none) -> OK; Obs (none) -> wes
- C_RST1: renamed from C3; value 0.1uF/50v(10%) -> 0.1uF 10V; # (none) -> CGA3E2X7R1H104K080AA; Group (none) -> Reset; Id CGA3E2X7R1H104K080AA -> (none); Mouser (none) -> OK
- C_SER1: renamed from C16; value 0.1uF -> 0.1uF 10V; # (none) -> CGA3E2X7R1H104K080AA; Group (none) -> Serial; Id CGA3E2X7R1H104K080AA -> (none); Mouser (none) -> OK
- C_SER2: renamed from C5; value 47pF -> 47pF 5V; # (none) -> CGA3E2C0G1H470J080AA; Group (none) -> Serial; Mouser (none) -> OK; Obs (none) -> wes
- C_SER3: renamed from C13; value 47pF -> 47pF 5V; # (none) -> CGA3E2C0G1H470J080AA; Group (none) -> Serial; Mouser (none) -> OK; Obs (none) -> wes
- C_SER4: renamed from C15; value 0.1uF -> 0.1uF 10V; # (none) -> CGA3E2X7R1H104K080AA; Group (none) -> Serial; Id CGA3E2X7R1H104K080AA -> (none); Mouser (none) -> OK
- C_SER5: renamed from C2; value 10uF/25v -> 10uF 12V 5mOhm; # (none) -> C1608X5R1E106M080AC; Group (none) -> Serial; Id C1608X5R1E106M080AC -> (none); Mouser (none) -> OK; Obs (none) -> wes
- C_SERVO1: renamed from C14; value 22uF/1mOhm -> 22uF 12V 1mOhm; # (none) -> C3225X7R1E226M250AB; Group (none) -> Servo; Id C1608JB1A226M080AC -> (none); Mouser (none) -> OK; Obs (none) -> wes
- C_STP1: renamed from C12; value 10uF/25v -> 10uF 12V 5mOhm; # (none) -> C1608X5R1E106M080AC; Group (none) -> 28BYJ-48 12V; Id C1608X5R1E106M080AC -> (none); Mouser (none) -> OK; Obs (none) -> wes
- C_WIFI1: renamed from C1; value 0.1uF/50v(10%) -> 0.1uF 10V; # (none) -> CGA3E2X7R1H104K080AA; Group (none) -> Wifi; Id CGA3E2X7R1H104K080AA -> (none); Mouser (none) -> OK
- D_HALL1: renamed from D9; value LED -> LED white; # (none) -> SMLD12WBN1W1; Group (none) -> Hall; Id B1931TW--20P000314U1930 -> (none); Mouser (none) -> OK
- D_NEMA1: renamed from D4; value LED -> LED white; # (none) -> SMLD12WBN1W1; Group (none) -> NEMA; Id B1931TW--20P000314U1930 -> (none); Mouser (none) -> OK
- D_NEMA2: renamed from D1; value LED -> LED white; # (none) -> SMLD12WBN1W1; Group (none) -> NEMA; Id B1931TW--20P000314U1930 -> (none); Mouser (none) -> OK
- D_POW1: renamed from D2; value LED -> LED white; # (none) -> SMLD12WBN1W1; Group (none) -> Latch power; Mouser (none) -> OK
- D_POW2: renamed from D11; value LED -> LED white; # (none) -> SMLD12WBN1W1; Group (none) -> Master power; Mouser (none) -> OK
- D_RX1, D_TX1: value LED -> LED white; # (none) -> SMLD12WBN1W1; Group (none) -> Serial; Mouser (none) -> OK
- D_SERVO1: renamed from D10; value LED -> LED white; # (none) -> SMLD12WBN1W1; Group (none) -> Servo; Id B1931TW--20P000314U1930 -> (none); Mouser (none) -> OK
- D_STP1: renamed from D5; value LED -> LED white; # (none) -> SMLD12WBN1W1; Group (none) -> 28BYJ-48 12V; Mouser (none) -> OK
- D_STP2: renamed from D6; value LED -> LED white; # (none) -> SMLD12WBN1W1; Group (none) -> 28BYJ-48 12V; Mouser (none) -> OK
- D_STP3: renamed from D7; value LED -> LED white; # (none) -> SMLD12WBN1W1; Group (none) -> 28BYJ-48 12V; Mouser (none) -> OK
- D_STP4: renamed from D8; value LED -> LED white; # (none) -> SMLD12WBN1W1; Group (none) -> 28BYJ-48 12V; Mouser (none) -> OK
- D_USB1: renamed from D_USBIN1; value LED -> LED white; # (none) -> SMLD12WBN1W1; Group (none) -> USB-C; Id B1931TW--20P000314U1930 -> (none); Mouser (none) -> OK
- FB_USB1: renamed from FB1; value 6V 750mA -> 40 Ohms @ 100 MHz 1 Power; # (none) -> MH2029-400Y; Group (none) -> USB-C; Id MH2029-400Y -> (none); Mouser (none) -> OK
- F_USB1: renamed from F1; value 6V 40A 750mA -> 6V 750mA; # (none) -> 0ZCK0075FF2E; Group (none) -> USB-C; Id 0ZCK0075FF2E -> (none); Mouser (none) -> OK
- H1, H2, H3, H4, H6: value MountingHole_Pad -> M3; # (none) -> -; Group (none) -> Pads; Mouser (none) -> OK
- JP_SER1: renamed from JP5; value SolderJumper_2_Bridged -> Bridged; # (none) -> -; Group (none) -> Serial; Mouser (none) -> OK
- JP_SER2: renamed from JP7; value SolderJumper_2_Bridged -> Bridged; # (none) -> -; Group (none) -> Serial; Mouser (none) -> OK
- JP_SER3: renamed from JP4; value SolderJumper_2_Bridged -> Bridged; # (none) -> -; Group (none) -> Serial; Mouser (none) -> OK
- JP_SER4: renamed from JP6; value SolderJumper_2_Bridged -> Bridged; # (none) -> -; Group (none) -> Serial; Mouser (none) -> OK
- J_28byj-48-12v_1: # (none) -> M20-9990546; Group (none) -> 28BYJ-48 12V; Mouser (none) -> OK
- J_HALL1: # (none) -> M20-9990346; Group (none) -> Hall; Mouser (none) -> OK
- J_LEDE1: renamed from J_LED_END1; # (none) -> M20-9990245; Group (none) -> LED end; Mouser (none) -> OK
- J_LEDP1: renamed from J_LED_PRESS1; # (none) -> M20-9990245; Group (none) -> LED press; Mouser (none) -> OK
- J_NEMA1: renamed from J_17HS4023_1; footprint Connector_PinHeader_2.54mm:PinHeader_1x04_P2.54mm_Vertical -> Connector_PinHeader_2.54mm:PinHeader_1x04_P2.54mm_Horizontal; # (none) -> M20-9750446; Group (none) -> NEMA; Mouser (none) -> OK
- J_OLED1: # (none) -> M20-9770446; Group (none) -> OLED display; Mouser (none) -> OK
- J_POW1: renamed from J_masterpower1; # (none) -> DCJ200-10-A-K1-K; Group (none) -> Master power; Id DCJ200-10-A-K1-K -> (none); Mouser (none) -> OK
- J_SERVO1: # (none) -> M20-9990346; Group (none) -> Servo; Mouser (none) -> OK
- J_USB1: renamed from J1; # (none) -> USB4105-GF-A; Group (none) -> USB-C; MANUFACTURER GCT -> (none); MAXIMUM_PACKAGE_HEIGHT 3.31 mm -> (none); Mouser (none) -> OK; PARTREV A3 -> (none); STANDARD Manufacturer Recommendations -> (none)
- L1: renamed from 11uH/15.8mOhm1; value SRP6060FA-100M -> 11uH/15.8mOhm1; # (none) -> SRP6060FA-100M; Group (none) -> 6V power; Mouser (none) -> OK
- Q_AUTO1: renamed from Q1; value SS8050-G -> SS8050; # (none) -> MMSS8050-L-TP; Category Discrete Semiconductor Products -> (none); DK_Datasheet_Link https://www.mccsemi.com/pdf/Products/MMSS8050(SOT-23).pdf -> (none); DK_Detail_Page /product-detail/en/micro-commercial-co/MMSS8050-H-TP/MMSS80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 -> (none); Digi-Key_PN MMSS8050-H-TPMSCT-ND -> (none); Family Transistors - Bipolar (BJT) - Single -> (none); Group (none) -> Autoboot; Id SS8050-G -> (none); MPN MMSS8050-H-TP -> (none); Manufacturer Micro Commercial Co -> (none); Mouser (none) -> OK; Status Active -> (none)
- Q_AUTO2: renamed from Q2; value SS8050-G -> SS8050; # (none) -> MMSS8050-L-TP; Category Discrete Semiconductor Products -> (none); DK_Datasheet_Link https://www.mccsemi.com/pdf/Products/MMSS8050(SOT-23).pdf -> (none); DK_Detail_Page /product-detail/en/micro-commercial-co/MMSS8050-H-TP/MMSS80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 -> (none); Digi-Key_PN MMSS8050-H-TPMSCT-ND -> (none); Family Transistors - Bipolar (BJT) - Single -> (none); Group (none) -> Autoboot; Id SS8050-G -> (none); MPN MMSS8050-H-TP -> (none); Manufacturer Micro Commercial Co -> (none); Mouser (none) -> OK; Status Active -> (none)
- Q_HALL1: # (none) -> BSS138W-7-F; Group (none) -> Hall; Id BSS138W-TP -> (none); Mouser (none) -> OK
- Q_POW1: renamed from Q3; value AO3401A -> IRLML6302TRPBF; # (none) -> IRLML6302TRPBF; Category Discrete Semiconductor Products -> (none); DK_Datasheet_Link http://aosmd.com/res/data_sheets/AO3401A.pdf -> (none); DK_Detail_Page /product-detail/en/alpha-omega-semiconductor-inc/AO3401A/78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 -> (none); Digi-Key_PN 785-1001-1-ND -> (none); Family Transistors - FETs, MOSFETs - Single -> (none); Group (none) -> Latch power; MPN AO3401A -> (none); Manufacturer Alpha & Omega Semiconductor Inc. -> (none); Mouser (none) -> OK; Obs (none) -> wes SI2303CDS-T1-BE3 ?? Id - Continuous Drain Current; Status Active -> (none)
- Q_POW2: renamed from Q4; value 2SC4213 -> MMBT3904,215; # (none) -> MMBT3904,215; Group (none) -> Latch power; Mouser (none) -> OK; Obs (none) -> wes
- Q_POW3: renamed from Q5; value 2SC4213 -> MMBT3904,215; # (none) -> MMBT3904,215; Group (none) -> Latch power; Mouser (none) -> OK; Obs (none) -> wes
- Q_SERVO1: # (none) -> BSS138W-7-F; Group (none) -> Servo; Id BSS138W-TP -> (none); Mouser (none) -> OK
- R_AUTO1: renamed from R7; value 10K(5%) -> 10K (5%); footprint Resistor_SMD:R_0603_1608Metric -> Resistor_SMD:R_0603_1608Metric_Pad0.98x0.95mm_HandSolder; # (none) -> CHP0603AFX-1002ELF; Group (none) -> Autoboot; Id ERJ-3EKF1002V -> (none); Mouser (none) -> OK; Obs (none) -> wes
- R_AUTO2: renamed from R8; value 10K(5%) -> 10K (5%); footprint Resistor_SMD:R_0603_1608Metric -> Resistor_SMD:R_0603_1608Metric_Pad0.98x0.95mm_HandSolder; # (none) -> CHP0603AFX-1002ELF; Group (none) -> Autoboot; Id ERJ-3EKF1002V -> (none); Mouser (none) -> OK; Obs (none) -> wes
- R_ENA1: renamed from R1; value 10K(5%) -> 10K (5%); footprint Resistor_SMD:R_0603_1608Metric -> Resistor_SMD:R_0603_1608Metric_Pad0.98x0.95mm_HandSolder; # (none) -> CHP0603AFX-1002ELF; Group (none) -> Enable; Id ERJ-3EKF1002V -> (none); Mouser (none) -> OK; Obs (none) -> wes
- R_HALL1: renamed from R10; value 10K -> 10K (5%); footprint Resistor_SMD:R_0603_1608Metric -> Resistor_SMD:R_0603_1608Metric_Pad0.98x0.95mm_HandSolder; # (none) -> CHP0603AFX-1002ELF; Group (none) -> Hall; Id ERJ-3EKF1002V -> (none); Mouser (none) -> OK; Obs (none) -> wes
- R_HALL2: renamed from R11; value 10K -> 10K (5%); footprint Resistor_SMD:R_0603_1608Metric -> Resistor_SMD:R_0603_1608Metric_Pad0.98x0.95mm_HandSolder; # (none) -> CHP0603AFX-1002ELF; Group (none) -> Hall; Id ERJ-3EKF1002V -> (none); Mouser (none) -> OK; Obs (none) -> wes
- R_HALL3: renamed from R24; value 47R -> 27R; footprint Resistor_SMD:R_0603_1608Metric -> Resistor_SMD:R_0603_1608Metric_Pad0.98x0.95mm_HandSolder; # (none) -> CMP0603-FX-27R0ELF; Group (none) -> Hall; Mouser (none) -> OK; Obs (none) -> wes
- R_LEDE1: renamed from R21; value 47R -> 27R; footprint Resistor_SMD:R_0603_1608Metric -> Resistor_SMD:R_0603_1608Metric_Pad0.98x0.95mm_HandSolder; # (none) -> CMP0603-FX-27R0ELF; Group (none) -> LED end; Mouser (none) -> OK; Obs (none) -> wes
- R_LEDP1: renamed from R20; value 47R -> 27R; footprint Resistor_SMD:R_0603_1608Metric -> Resistor_SMD:R_0603_1608Metric_Pad0.98x0.95mm_HandSolder; # (none) -> CMP0603-FX-27R0ELF; Group (none) -> LED press; Mouser (none) -> OK; Obs (none) -> wes
- R_NEMA1: renamed from R26; value 47R -> 27R; footprint Resistor_SMD:R_0603_1608Metric -> Resistor_SMD:R_0603_1608Metric_Pad0.98x0.95mm_HandSolder; # (none) -> CMP0603-FX-27R0ELF; Group (none) -> NEMA; Mouser (none) -> OK; Obs (none) -> wes
- R_NEMA2: renamed from R27; value 47R -> 27R; footprint Resistor_SMD:R_0603_1608Metric -> Resistor_SMD:R_0603_1608Metric_Pad0.98x0.95mm_HandSolder; # (none) -> CMP0603-FX-27R0ELF; Group (none) -> NEMA; Mouser (none) -> OK; Obs (none) -> wes
- R_POW1: renamed from R28; # (none) -> CR0603-JW-431ELF; Group (none) -> Latch power; Id ERJ-PA3F4300V -> (none); Mouser (none) -> OK; Obs (none) -> wes
- R_POW2: renamed from R29; # (none) -> CHP0603AFX-1003ELF; Group (none) -> Latch power; Id ERJ-PA3J101V -> (none); Mouser (none) -> OK; Obs (none) -> wes
- R_POW3: renamed from R30; # (none) -> CHP0603AFX-1003ELF; Group (none) -> Latch power; Id ERJ-PA3J101V -> (none); Mouser (none) -> OK; Obs (none) -> wes
- R_POW4: renamed from R31; # (none) -> CMP0603AFX-1004ELF; Group (none) -> Latch power; Id ERJ-PA3J101V -> (none); Mouser (none) -> OK; Obs (none) -> wes
- R_POW5: renamed from R32; # (none) -> CHP0603AFX-1003ELF; Group (none) -> Latch power; Id ERJ-PA3J101V -> (none); Mouser (none) -> OK; Obs (none) -> wes
- R_POW6: renamed from R2; # (none) -> CR0603-JW-431ELF; Group (none) -> Master power; Id ERJ-PA3F4300V -> (none); Mouser (none) -> OK; Obs (none) -> wes
- R_POW_FBT1: renamed from R_FBT1; # (none) -> CHP0603AFX-1003ELF; Group (none) -> 6V power; Id ERJ-PA3J101V -> (none); Mouser (none) -> OK; Obs (none) -> wes
- R_POW_FFB1: renamed from R_FFB1; # (none) -> CRCW060311K0JNEAHP; Group (none) -> 6V power; Id ERJ-PA3J101V -> (none); Mouser (none) -> OK; Obs (none) -> wes
- R_RST1: renamed from R5; value 10K(5%) -> 10K (5%); footprint Resistor_SMD:R_0603_1608Metric -> Resistor_SMD:R_0603_1608Metric_Pad0.98x0.95mm_HandSolder; # (none) -> CHP0603AFX-1002ELF; Group (none) -> Reset; Id ERJ-3EKF1002V -> (none); Mouser (none) -> OK; Obs (none) -> wes
- R_RX1: renamed from R22; value 47R -> 27R; footprint Resistor_SMD:R_0603_1608Metric -> Resistor_SMD:R_0603_1608Metric_Pad0.98x0.95mm_HandSolder; # (none) -> CMP0603-FX-27R0ELF; Group (none) -> Serial; Mouser (none) -> OK; Obs (none) -> wes
- R_SER1: renamed from R14; # (none) -> CMP0603-FX-27R0ELF; Group (none) -> Serial; Mouser (none) -> OK; Obs (none) -> wes
- R_SER2: renamed from R19; # (none) -> CMP0603-FX-27R0ELF; Group (none) -> Serial; Mouser (none) -> OK; Obs (none) -> wes
- R_SERVO1: renamed from R12; value 10K -> 10K (5%); footprint Resistor_SMD:R_0603_1608Metric -> Resistor_SMD:R_0603_1608Metric_Pad0.98x0.95mm_HandSolder; # (none) -> CHP0603AFX-1002ELF; Group (none) -> Servo; Id ERJ-3EKF1002V -> (none); Mouser (none) -> OK; Obs (none) -> wes
- R_SERVO2: renamed from R13; value 10K -> 10K (5%); footprint Resistor_SMD:R_0603_1608Metric -> Resistor_SMD:R_0603_1608Metric_Pad0.98x0.95mm_HandSolder; # (none) -> CHP0603AFX-1002ELF; Group (none) -> Servo; Id ERJ-3EKF1002V -> (none); Mouser (none) -> OK; Obs (none) -> wes
- R_SERVO3: renamed from R25; value 47R -> 27R; footprint Resistor_SMD:R_0603_1608Metric -> Resistor_SMD:R_0603_1608Metric_Pad0.98x0.95mm_HandSolder; # (none) -> CMP0603-FX-27R0ELF; Group (none) -> Servo; Mouser (none) -> OK; Obs (none) -> wes
- R_STP1: renamed from R15; footprint Resistor_SMD:R_0603_1608Metric -> Resistor_SMD:R_0603_1608Metric_Pad0.98x0.95mm_HandSolder; # (none) -> CR0603-JW-431ELF; Group (none) -> 28BYJ-48 12V; Id ERJ-PA3F4300V -> (none); Mouser (none) -> OK; Obs (none) -> wes
- R_STP2: renamed from R16; footprint Resistor_SMD:R_0603_1608Metric -> Resistor_SMD:R_0603_1608Metric_Pad0.98x0.95mm_HandSolder; # (none) -> CR0603-JW-431ELF; Group (none) -> 28BYJ-48 12V; Id ERJ-PA3F4300V -> (none); Mouser (none) -> OK; Obs (none) -> wes
- R_STP3: renamed from R17; footprint Resistor_SMD:R_0603_1608Metric -> Resistor_SMD:R_0603_1608Metric_Pad0.98x0.95mm_HandSolder; # (none) -> CR0603-JW-431ELF; Group (none) -> 28BYJ-48 12V; Id ERJ-PA3F4300V -> (none); Mouser (none) -> OK; Obs (none) -> wes
- R_STP4: renamed from R18; footprint Resistor_SMD:R_0603_1608Metric -> Resistor_SMD:R_0603_1608Metric_Pad0.98x0.95mm_HandSolder; # (none) -> CR0603-JW-431ELF; Group (none) -> 28BYJ-48 12V; Id ERJ-PA3F4300V -> (none); Mouser (none) -> OK; Obs (none) -> wes
- R_TX1: renamed from R23; value 47R -> 27R; footprint Resistor_SMD:R_0603_1608Metric -> Resistor_SMD:R_0603_1608Metric_Pad0.98x0.95mm_HandSolder; # (none) -> CMP0603-FX-27R0ELF; Group (none) -> Serial; Mouser (none) -> OK; Obs (none) -> wes
- R_USB1: renamed from R3; value 5.1K(10%) -> 5.1K (10%); # (none) -> CR0603-FX-5101ELF; Group (none) -> USB-C; Id ERJ-3EKF5101V -> (none); Mouser (none) -> OK; Obs (none) -> wes
- R_USB2: renamed from R9; value 5.1K(10%) -> 5.1K (10%); # (none) -> CR0603-FX-5101ELF; Group (none) -> USB-C; Id ERJ-3EKF5101V -> (none); Mouser (none) -> OK; Obs (none) -> wes
- R_USB3: renamed from R6; # (none) -> CHP0603AFX-1000ELF; Group (none) -> USB-C; Id ERJ-PA3J101V -> (none); Mouser (none) -> OK; Obs (none) -> wes
- R_WIFI1: renamed from R4; # (none) -> CHP0603AFX-1002ELF; Group (none) -> Wifi; Id ERJ-3EKF1002V -> (none); Mouser (none) -> OK; Obs (none) -> wes
- SW_ENA1: renamed from SW2; # (none) -> B3FS-1000; Group (none) -> Enable; Mouser (none) -> OK
- SW_POW1: renamed from SW4; # (none) -> B3FS-1000; Group (none) -> Latch power; Mouser (none) -> OK
- SW_RST1: renamed from SW1; # (none) -> B3FS-1000; Group (none) -> Reset; Mouser (none) -> OK
- SW_WIFI1: renamed from SW3; # (none) -> B3FS-1000; Group (none) -> Wifi; Mouser (none) -> OK
- TP_12v1, TP_3.3v1, TP_5v1, TP_6v1, TP_GND2, TP_GND3: # (none) -> -; Group (none) -> Pads; Mouser (none) -> OK
- TP_CTS1, TP_DTR1, TP_GND1, TP_RX1, TP_TX1, TP_VCC_3.3V1: # (none) -> -; Group (none) -> External flash; Mouser (none) -> OK
- U_MCU1: renamed from U4; # (none) -> ESP32-WROOM-32D-N4; Group (none) -> MCU; Mouser (none) -> OK
- U_POW1: renamed from U5; # (none) -> TPS54302; Group (none) -> 6V power; Mouser (none) -> N; Obs (none) -> wes / alternative TPS5430MDDAREP not dropin
- U_POW2: renamed from U2; value AZ1117I-3.3 -> AZ1117CH-3.3TRG1; # (none) -> AZ1117CH-3.3TRG1; Category Integrated Circuits (ICs) -> (none); DK_Datasheet_Link https://www.diodes.com/assets/Datasheets/AZ1117C.pdf -> (none); DK_Detail_Page /product-detail/en/diodes-incorporated/AZ1117CH-3.3TRG1/AZ1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 -> (none); Digi-Key_PN AZ1117CH-3.3TRG1DICT-ND -> (none); Family PMIC - Voltage Regulators - Linear -> (none); Group (none) -> 3V3 power; Id AZ1117IH-3.3TRG1 -> (none); MPN AZ1117CH-3.3TRG1 -> (none); Manufacturer Diodes Incorporated -> (none); Mouser (none) -> OK; Status Active -> (none)
- U_SER1: renamed from U3; value FT231XS -> FT231XS-R; # (none) -> FT231XS-R; Group (none) -> Serial; Mouser (none) -> OK
- U_STP1: renamed from U6; # (none) -> ULN2003ADR2G; Group (none) -> 28BYJ-48 12V; Id ULN2003ADR2G -> (none); Mouser (none) -> OK
- U_USB1: renamed from U1; # (none) -> USB6B1RL; Group (none) -> USB-C; Id USB6B1 -> (none); Mouser (none) -> OK
Other:
- added sheet 6V Power (6vpower.kicad_sch)
- note added: "BOOT"
- note removed: "BOOT & RESET"
- note removed: "hall: voltage divider"
- note removed: "servo, mosfet"
- moved on the sheet: C_POW3, C_POW_6V_FF1, C_POW_BST1, C_POW_IN1, C_POW_IN2, C_POW_IN3, C_POW_OUT1, C_POW_OUT2, C_POW_OUT3, C_POW_OUT4, C_POW_OUT5, C_SER4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

Commit message: visual identity on silk and exposed copper layers
Parts:
- J_HALL1: value Conn_01x03_Male -> Conn_01x03_Female; footprint Connector_PinHeader_2.54mm:PinHeader_1x03_P2.54mm_Vertical -> Connector_PinSocket_2.54mm:PinSocket_1x03_P2.54mm_Vertical; # M20-9990346 -> M20-7820346
Changed lines of the file:
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@@
       (effects (font (size 1.27 1.27)) (justify right))
     )
-    (property "Value" "Conn_01x03_Male" (id 1) (at 93.98 274.3199 0)
+    (property "Value" "Conn_01x03_Female" (id 1) (at 93.98 274.3199 0)
       (effects (font (size 1.27 1.27)) (justify right))
     )
-    (property "Footprint" "Connector_PinHeader_2.54mm:PinHeader_1x03_P2.54mm_Vertical" (id 2) (at 95.25 273.05 0)
+    (property "Footprint" "Connector_PinSocket_2.54mm:PinSocket_1x03_P2.54mm_Vertical" (id 2) (at 95.25 273.05 0)
       (effects (font (size 1.27 1.27)) hide)
     )
-    (property "Datasheet" "https://br.mouser.com/datasheet/2/181/M20-999-1218971.pdf" (id 3) (at 95.25 273.05 0)
+    (property "Datasheet" "https://br.mouser.com/datasheet/2/181/M20-782-1220556.pdf" (id 3) (at 95.25 273.05 0)
       (effects (font (size 1.27 1.27)) hide)
     )
-    (property "#" "M20-9990346" (id 6) (at 95.25 273.05 0)
+    (property "#" "M20-7820346" (id 6) (at 95.25 273.05 0)
       (effects (font (size 1.27 1.27)) hide)
     )
@@
     )
     (property "#" "CMP0603-FX-27R0ELF" (id 4) (at 199.39 274.32 0)
-      (effects (font (size 1.27 1.27) italic) (justify left))
+      (effects (font (size 1.27 1.27) italic) (justify left) hide)
     )
     (property "Description" "LED series resistor" (id 5) (at 200.66 271.78 90)
@@
     )
     (property "#" "CMP0603-FX-27R0ELF" (id 4) (at 146.05 274.32 0)
-      (effects (font (size 1.27 1.27) italic) (justify left))
+      (effects (font (size 1.27 1.27) italic) (justify left) hide)
     )
     (property "Description" "LED series resistor" (id 5) (at 147.32 271.78 90)
@@
     )
     (path "/20a74162-9bd6-4db0-9556-2d7b4949d5a0"
-      (reference "J_HALL1") (unit 1) (value "Conn_01x03_Male") (footprint "Connector_PinHeader_2.54mm:PinHeader_1x03_P2.54mm_Vertical")
+      (reference "J_HALL1") (unit 1) (value "Conn_01x03_Female") (footprint "Connector_PinSocket_2.54mm:PinSocket_1x03_P2.54mm_Vertical")
     )
     (path "/9aa1a152-e0a0-4fc5-882c-06dcd76cbb55"

Commit message: hierarchical sheets and overall organization
Parts:
- removed A_NEMA1: 8+8 pin, SnapEDA Library:Pololu_Breakout-16_15.2x20.3mm, symbol Driver_Motor:Pololu_Breakout_A4988
- removed C_ENA1, C_MCU1, C_RST1, C_SER1, C_SER4, C_WIFI1: 0.1uF 10V, Capacitor_SMD:C_0603_1608Metric_Pad1.08x0.95mm_HandSolder, symbol Device:C
- removed C_MCU2, C_POW2, C_POW3: 22uF 12V 1mOhm, Capacitor_SMD:C_0603_1608Metric_Pad1.08x0.95mm_HandSolder, symbol Device:C
- removed C_NEMA1: 100uF 25V, Capacitor_SMD:CP_Elec_6.3x5.9, symbol Device:C_Polarized
- removed C_NEMA2, C_POW1, C_SER5, C_STP1: 10uF 12V 5mOhm, Capacitor_SMD:C_0603_1608Metric_Pad1.08x0.95mm_HandSolder, symbol Device:C
- removed C_POW_6V_FF1: 82pF 6V 0Ohm, Capacitor_SMD:C_0603_1608Metric_Pad1.08x0.95mm_HandSolder, symbol Device:C
- removed C_POW_BST1: 100nF 6V 64mOhm, Capacitor_SMD:C_0603_1608Metric_Pad1.08x0.95mm_HandSolder, symbol Device:C
- removed C_POW_IN1, C_POW_IN2, C_POW_IN3: 10uF 12V 5mOhm, Capacitor_SMD:C_1210_3225Metric_Pad1.33x2.70mm_HandSolder, symbol Device:C
- removed C_POW_OUT1, C_POW_OUT2, C_POW_OUT3, C_POW_OUT4, C_POW_OUT5, C_SERVO1: 22uF 12V 1mOhm, Capacitor_SMD:C_1210_3225Metric_Pad1.33x2.70mm_HandSolder, symbol Device:C
- removed C_SER2, C_SER3: 47pF 5V, Capacitor_SMD:C_0603_1608Metric_Pad1.08x0.95mm_HandSolder, symbol Device:C
- removed D_HALL1, D_NEMA1, D_NEMA2, D_POW1, D_POW2, D_RX1, D_SERVO1, D_STP1, D_STP2, D_STP3, D_STP4, D_TX1, D_USB1: LED white, LED_SMD:LED_0603_1608Metric_Pad1.05x0.95mm_HandSolder, symbol Device:LED
- removed FB_USB1: 40 Ohms @ 100 MHz 1 Power, Inductor_SMD:L_0805_2012Metric_Pad1.05x1.20mm_HandSolder, symbol Device:FerriteBead
- removed F_USB1: 6V 750mA, Fuse:Fuse_0805_2012Metric_Pad1.15x1.40mm_HandSolder, symbol Device:Polyfuse
- removed H1, H2, H3, H4, H6: M3, MountingHole:MountingHole_3.2mm_M3_Pad_Via, symbol Mechanical:MountingHole_Pad
- removed JP_SER1, JP_SER2, JP_SER3, JP_SER4: Bridged, Jumper:SolderJumper-2_P1.3mm_Bridged2Bar_Pad1.0x1.5mm, symbol Jumper:SolderJumper_2_Bridged
- removed J_28byj-48-12v_1: Conn_01x05_Male, Connector_PinHeader_2.54mm:PinHeader_1x05_P2.54mm_Vertical, symbol Connector:Conn_01x05_Male
- removed J_HALL1: Conn_01x03_Female, Connector_PinSocket_2.54mm:PinSocket_1x03_P2.54mm_Vertical, symbol Connector:Conn_01x03_Male
- removed J_LEDE1, J_LEDP1: Conn_01x02_Male, Connector_PinHeader_2.54mm:PinHeader_1x02_P2.54mm_Vertical, symbol Connector:Conn_01x02_Male
- removed J_NEMA1: Conn_01x04_Male, Connector_PinHeader_2.54mm:PinHeader_1x04_P2.54mm_Horizontal, symbol Connector:Conn_01x04_Male
- removed J_OLED1: Conn_01x04_Male, Connector_PinHeader_2.54mm:PinHeader_1x04_P2.54mm_Vertical, symbol Connector:Conn_01x04_Male
- removed J_POW1: Barrel_Jack_Switch, SnapEDA Library:BarrelJack_GCT_DCJ200-10-A_Horizontal, symbol Connector:Barrel_Jack_Switch
- removed J_SERVO1: Conn_01x03_Male, Connector_PinHeader_2.54mm:PinHeader_1x03_P2.54mm_Vertical, symbol Connector:Conn_01x03_Male
- removed J_USB1: USB4105-GF-A, SnapEDA Library:GCT_USB4105-GF-A, symbol USB4105-GF-A:USB4105-GF-A
- removed L1: 11uH/15.8mOhm1, SRP6060FA:SRP6060FA-4R7M, symbol Device:L
- removed Q_AUTO1, Q_AUTO2: SS8050, Package_TO_SOT_SMD:SOT-23, symbol dk_Transistors-Bipolar-BJT-Single:MMSS8050-H-TP
- removed Q_HALL1, Q_SERVO1: BSS138, Package_TO_SOT_SMD:SOT-23, symbol Transistor_FET:BSS138
- removed Q_POW1: IRLML6302TRPBF, Package_TO_SOT_SMD:SOT-23, symbol dk_Transistors-FETs-MOSFETs-Single:AO3401A
- removed Q_POW2, Q_POW3: MMBT3904,215, Package_TO_SOT_SMD:SOT-23, symbol Transistor_BJT:2SC4213
- removed R_AUTO1, R_AUTO2, R_ENA1, R_HALL1, R_HALL2, R_RST1, R_SERVO1, R_SERVO2: 10K (5%), Resistor_SMD:R_0603_1608Metric_Pad0.98x0.95mm_HandSolder, symbol Device:R
- removed R_HALL3, R_LEDE1, R_LEDP1, R_NEMA1, R_NEMA2, R_RX1, R_SER1, R_SER2, R_SERVO3, R_TX1: 27R, Resistor_SMD:R_0603_1608Metric_Pad0.98x0.95mm_HandSolder, symbol Device:R
- removed R_POW1, R_POW6, R_STP1, R_STP2, R_STP3, R_STP4: 430R, Resistor_SMD:R_0603_1608Metric_Pad0.98x0.95mm_HandSolder, symbol Device:R
- removed R_POW2, R_POW3, R_POW5, R_POW_FBT1: 100K, Resistor_SMD:R_0603_1608Metric_Pad0.98x0.95mm_HandSolder, symbol Device:R
- removed R_POW4: 1M, Resistor_SMD:R_0603_1608Metric_Pad0.98x0.95mm_HandSolder, symbol Device:R
- removed R_POW_FFB1: 11K, Resistor_SMD:R_0603_1608Metric_Pad0.98x0.95mm_HandSolder, symbol Device:R
- removed R_USB1, R_USB2: 5.1K (10%), Resistor_SMD:R_0603_1608Metric_Pad0.98x0.95mm_HandSolder, symbol Device:R
- removed R_USB3: 100R, Resistor_SMD:R_0603_1608Metric_Pad0.98x0.95mm_HandSolder, symbol Device:R
- removed R_WIFI1: 10K(5%), Resistor_SMD:R_0603_1608Metric_Pad0.98x0.95mm_HandSolder, symbol Device:R
- removed SW_ENA1, SW_POW1, SW_RST1, SW_WIFI1: B3FS-1000, b3fs:B3FS-1000, symbol 2022-07-12_23-59-33:B3FS-1000
- removed TP_12v1, TP_3.3v1, TP_5v1, TP_6v1, TP_CTS1, TP_DTR1, TP_GND1, TP_GND2, TP_GND3, TP_RX1, TP_TX1, TP_VCC_3.3V1: TestPoint, TestPoint:TestPoint_Pad_D1.0mm, symbol Connector:TestPoint
- removed U_MCU1: ESP32-WROOM-32, RF_Module:ESP32-WROOM-32, symbol RF_Module:ESP32-WROOM-32
- removed U_POW1: TPS54302, Package_TO_SOT_SMD:SOT-23-6, symbol Regulator_Switching:TPS54302
- removed U_POW2: AZ1117CH-3.3TRG1, Package_TO_SOT_SMD:SOT-223, symbol dk_PMIC-Voltage-Regulators-Linear:AZ1117CH-3_3TRG1
- removed U_SER1: FT231XS-R, Package_SO:SSOP-20_3.9x8.7mm_P0.635mm, symbol Interface_USB:FT231XS
- removed U_STP1: ULN2003, Package_SO:SOIC-16W_5.3x10.2mm_P1.27mm, symbol Transistor_Array:ULN2003
- removed U_USB1: USB6B1, Package_SO:SOIC-8_3.9x4.9mm_P1.27mm, symbol Power_Protection:USB6B1
Connections:
- no-connect marks 30 -> 0
Other:
- added sheet 12V Power (power12v.kicad_sch)
- added sheet 3V3 Power (power3v3.kicad_sch)
- added sheet Boot (boot.kicad_sch)
- added sheet Char Stepper (charstepper.kicad_sch)
- added sheet Connectors (connectors.kicad_sch)
- added sheet External Flashing (extflashing.kicad_sch)
- added sheet Feed Stepper (feedstepper.kicad_sch)
- added sheet Level Shift (levelshift.kicad_sch)
- added sheet MCU (mcu.kicad_sch)
- added sheet Serial (serial.kicad_sch)
- added sheet Test Pads (testpads.kicad_sch)
- added sheet USB-C 2.0 (usb.kicad_sch)
- added sheet Wifi Reset (wifireset.kicad_sch)
- sheet 6V Power: file 6vpower.kicad_sch -> power6v.kicad_sch
- note added: "EN / BOOT"
- note added: "EXT FLASHING"
- note added: "POWER"
- note added: "SERIAL"
- note added: "TEST PADS"
- note removed: "12V POWER"
- note removed: "3.3V POWER"
- note removed: "6V POWER"
- note removed: "6V POWER: BUCK"
- note removed: "BOOT"
- note removed: "EXTERNAL FLASHING"
- note removed: "FTDI"
- note removed: "LATCH POWER"
- note removed: "PADS / TESTING"
