File: _electronic/KiCad/boot.kicad_sch (KiCad schematic)
At the start: 10 parts

Commit message: external flashing header
Other:
- note added: "Auto program DTR RTS --> EN IO0 1 1 1 1 0 0 1 1 1 0 0 1 0 1 1 0"
Changed lines of the file:
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@@
   (junction (at 182.88 81.28) (diameter 0) (color 0 0 0 0)
   )
+  (wire (pts (xy 153.67 118.11) (xy 153.67 146.05))
+    (stroke (width 0) (type default) (color 0 0 0 0))
+  )
+  (wire (pts (xy 100.33 115.57) (xy 100.33 105.41))
+    (stroke (width 0) (type default) (color 0 0 0 0))
+  )
+  (wire (pts (xy 165.1 96.52) (xy 165.1 95.25))
+    (stroke (width 0) (type default) (color 0 0 0 0))
+  )
+  (wire (pts (xy 189.23 66.04) (xy 189.23 69.85))
+    (stroke (width 0) (type default) (color 0 0 0 0))
+  )
+  (wire (pts (xy 182.88 130.81) (xy 182.88 146.05))
+    (stroke (width 0) (type default) (color 0 0 0 0))
+  )
+  (wire (pts (xy 165.1 68.58) (xy 165.1 69.85))
+    (stroke (width 0) (type default) (color 0 0 0 0))
+  )
+  (wire (pts (xy 153.67 68.58) (xy 162.56 68.58))
+    (stroke (width 0) (type default) (color 0 0 0 0))
+  )
+  (wire (pts (xy 189.23 127) (xy 189.23 130.81))
+    (stroke (width 0) (type default) (color 0 0 0 0))
+  )
+  (wire (pts (xy 165.1 146.05) (xy 182.88 146.05))
+    (stroke (width 0) (type default) (color 0 0 0 0))
+  )
+  (wire (pts (xy 182.88 118.11) (xy 182.88 130.81))
+    (stroke (width 0) (type default) (color 0 0 0 0))
+  )
+  (wire (pts (xy 97.79 97.79) (xy 97.79 107.95))
+    (stroke (width 0) (type default) (color 0 0 0 0))
+  )
+  (wire (pts (xy 189.23 100.33) (xy 189.23 91.44))
+    (stroke (width 0) (type default) (color 0 0 0 0))
+  )
+  (wire (pts (xy 182.88 130.81) (xy 189.23 130.81))
+    (stroke (width 0) (type default) (color 0 0 0 0))
+  )
+  (wire (pts (xy 153.67 68.58) (xy 153.67 96.52))
+    (stroke (width 0) (type default) (color 0 0 0 0))
+  )
+  (wire (pts (xy 189.23 133.35) (xy 189.23 130.81))
+    (stroke (width 0) (type default) (color 0 0 0 0))
+  )
+  (wire (pts (xy 120.65 90.17) (xy 120.65 92.71))
+    (stroke (width 0) (type default) (color 0 0 0 0))
+  )
+  (wire (pts (xy 182.88 68.58) (xy 182.88 81.28))
+    (stroke (width 0) (type default) (color 0 0 0 0))
+  )
+  (wire (pts (xy 165.1 68.58) (xy 182.88 68.58))
+    (stroke (width 0) (type default) (color 0 0 0 0))
+  )
   (wire (pts (xy 120.65 107.95) (xy 120.65 110.49))
     (stroke (width 0) (type default) (color 0 0 0 0))
   )
-  (wire (pts (xy 153.67 118.11) (xy 153.67 146.05))
-    (stroke (width 0) (type default) (color 0 0 0 0))
-  )
-  (wire (pts (xy 100.33 115.57) (xy 100.33 105.41))
-    (stroke (width 0) (type default) (color 0 0 0 0))
-  )
-  (wire (pts (xy 165.1 96.52) (xy 165.1 95.25))
-    (stroke (width 0) (type default) (color 0 0 0 0))
-  )
-  (wire (pts (xy 189.23 66.04) (xy 189.23 69.85))
-    (stroke (width 0) (type default) (color 0 0 0 0))
-  )
-  (wire (pts (xy 182.88 130.81) (xy 182.88 146.05))
-    (stroke (width 0) (type default) (color 0 0 0 0))
-  )
-  (wire (pts (xy 165.1 68.58) (xy 165.1 69.85))
-    (stroke (width 0) (type default) (color 0 0 0 0))
-  )
-  (wire (pts (xy 153.67 68.58) (xy 162.56 68.58))
-    (stroke (width 0) (type default) (color 0 0 0 0))
-  )
-  (wire (pts (xy 189.23 127) (xy 189.23 130.81))
-    (stroke (width 0) (type default) (color 0 0 0 0))
-  )
-  (wire (pts (xy 165.1 146.05) (xy 182.88 146.05))
-    (stroke (width 0) (type default) (color 0 0 0 0))
-  )
-  (wire (pts (xy 182.88 118.11) (xy 182.88 130.81))
-    (stroke (width 0) (type default) (color 0 0 0 0))
-  )
-  (wire (pts (xy 97.79 97.79) (xy 97.79 123.19))
-    (stroke (width 0) (type default) (color 0 0 0 0))
-  )
-  (wire (pts (xy 127 107.95) (xy 120.65 107.95))
-    (stroke (width 0) (type default) (color 0 0 0 0))
-  )
-  (wire (pts (xy 189.23 100.33) (xy 189.23 91.44))
-    (stroke (width 0) (type default) (color 0 0 0 0))
-  )
-  (wire (pts (xy 182.88 130.81) (xy 189.23 130.81))
-    (stroke (width 0) (type default) (color 0 0 0 0))
-  )
-  (wire (pts (xy 153.67 68.58) (xy 153.67 96.52))
-    (stroke (width 0) (type default) (color 0 0 0 0))
-  )
-  (wire (pts (xy 189.23 133.35) (xy 189.23 130.81))
-    (stroke (width 0) (type default) (color 0 0 0 0))
-  )
-  (wire (pts (xy 120.65 90.17) (xy 120.65 92.71))
-    (stroke (width 0) (type default) (color 0 0 0 0))
-  )
-  (wire (pts (xy 182.88 68.58) (xy 182.88 81.28))
-    (stroke (width 0) (type default) (color 0 0 0 0))
-  )
-  (wire (pts (xy 165.1 68.58) (xy 182.88 68.58))
-    (stroke (width 0) (type default) (color 0 0 0 0))
-  )
-  (wire (pts (xy 120.65 123.19) (xy 120.65 120.65))
+  (wire (pts (xy 120.65 120.65) (xy 120.65 123.19))
     (stroke (width 0) (type default) (color 0 0 0 0))
   )
@@
     (stroke (width 0) (type default) (color 0 0 0 0))
   )
-  (wire (pts (xy 97.79 123.19) (xy 120.65 123.19))
+  (wire (pts (xy 97.79 107.95) (xy 120.65 107.95))
     (stroke (width 0) (type default) (color 0 0 0 0))
   )
@@
     (stroke (width 0) (type default) (color 0 0 0 0))
   )
+  (wire (pts (xy 120.65 123.19) (xy 127 123.19))
+    (stroke (width 0) (type default) (color 0 0 0 0))
+  )
   (wire (pts (xy 120.65 105.41) (xy 120.65 102.87))
     (stroke (width 0) (type default) (color 0 0 0 0))
@@
   (wire (pts (xy 97.79 97.79) (xy 102.87 97.79))
     (stroke (width 0) (type default) (color 0 0 0 0))
+  )
+  (text "Auto program\n\nDTR RTS --> EN IO0\n 1    1         1  1\n 0    0         1  1\n 1    0         0  1\n 0    1         1  0"
+    (at 97.79 142.24 0)
+    (effects (font (size 1.27 1.27)) (justify left bottom))
   )
   (text "EN / BOOT" (at 114.3 45.72 0)
@@
     (effects (font (size 1.27 1.27)) (justify left))
   )
+  (hierarchical_label "RESET OUT" (shape input) (at 127 123.19 0)
+    (effects (font (size 1.27 1.27)) (justify left))
+  )
   (hierarchical_label "EN OUT" (shape input) (at 193.04 81.28 0)
     (effects (font (size 1.27 1.27)) (justify left))
@@
     (effects (font (size 1.27 1.27)) (justify right))
   )
-  (hierarchical_label "RESET OUT" (shape input) (at 127 107.95 0)
-    (effects (font (size 1.27 1.27)) (justify left))
-  )
   (hierarchical_label "3V3 IN" (shape input) (at 189.23 115.57 90)
     (effects (font (size 1.27 1.27)) (justify left))
@@
   (symbol (lib_id "Device:R") (at 106.68 97.79 90) (unit 1)
     (in_bom yes) (on_board yes)
-    (property "Reference" "R_AUTO1" (id 0) (at 106.68 91.44 90))
-    (property "Value" "10K (5%)" (id 1) (at 106.68 93.98 90))
+    (property "Reference" "R_AUTO1" (id 0) (at 106.68 95.25 90))
+    (property "Value" "10K (5%)" (id 1) (at 106.68 100.33 90))
     (property "Footprint" "Resistor_SMD:R_0603_1608Metric_Pad0.98x0.95mm_HandSolder" (id 2) (at 106.68 99.568 90)
       (effects (font (size 1.27 1.27)) hide)
@@
     (pin "2")
   )
-  (symbol (lib_id "dk_Transistors-Bipolar-BJT-Single:MMSS8050-H-TP") (at 118.11 115.57 0) (unit 1)
+  (symbol (lib_id "dk_Transistors-Bipolar-BJT-Single:MMSS8050-H-TP") (at 118.11 115.57 0) (mirror x) (unit 1)
     (in_bom yes) (on_board yes)
     (property "Reference" "Q_AUTO2" (id 0) (at 123.19 115.57 0)
       (effects (font (size 1.524 1.524)) (justify left))
     )
-    (property "Value" "SS8050" (id 1) (at 123.19 118.11 0)
+    (property "Value" "SS8050" (id 1) (at 123.19 113.03 0)
       (effects (font (size 1.524 1.524)) (justify left) hide)
     )
-    (property "Footprint" "Package_TO_SOT_SMD:SOT-23" (id 2) (at 123.19 110.49 0)
+    (property "Footprint" "Package_TO_SOT_SMD:SOT-23" (id 2) (at 123.19 120.65 0)
       (effects (font (size 1.524 1.524)) (justify left) hide)
     )
-    (property "Datasheet" "https://br.mouser.com/datasheet/2/258/MMSS8050_SOT_23_-1626440.pdf" (id 3) (at 123.19 107.95 0)
+    (property "Datasheet" "https://br.mouser.com/datasheet/2/258/MMSS8050_SOT_23_-1626440.pdf" (id 3) (at 123.19 123.19 0)
       (effects (font (size 1.524 1.524)) (justify left) hide)
     )
-    (property "#" "MMSS8050-L-TP" (id 13) (at 123.19 116.84 0)
+    (property "#" "MMSS8050-L-TP" (id 13) (at 123.19 114.3 0)
       (effects (font (size 1.27 1.27) italic) (justify left) hide)
     )
@@
   )
   (symbol (lib_id "Device:R") (at 106.68 115.57 90) (unit 1)
-    (in_bom yes) (on_board yes) (fields_autoplaced)
-    (property "Reference" "R_AUTO2" (id 0) (at 106.68 109.22 90))
-    (property "Value" "10K (5%)" (id 1) (at 106.68 111.76 90))
+    (in_bom yes) (on_board yes)
+    (property "Reference" "R_AUTO2" (id 0) (at 106.68 113.03 90))
+    (property "Value" "10K (5%)" (id 1) (at 106.68 118.11 90))
     (property "Footprint" "Resistor_SMD:R_0603_1608Metric_Pad0.98x0.95mm_HandSolder" (id 2) (at 106.68 117.348 90)
       (effects (font (size 1.27 1.27)) hide)

Commit message: revised IC packages, pins and footprints
Parts:
- Q_AUTO1, Q_AUTO2: footprint Package_TO_SOT_SMD:SOT-23 -> Package_TO_SOT_SMD:SOT-23_Handsoldering
Changed lines of the file:
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@@
       (effects (font (size 1.524 1.524)) (justify left) hide)
     )
-    (property "Footprint" "Package_TO_SOT_SMD:SOT-23" (id 2) (at 123.19 120.65 0)
+    (property "Footprint" "Package_TO_SOT_SMD:SOT-23_Handsoldering" (id 2) (at 123.19 120.65 0)
       (effects (font (size 1.524 1.524)) (justify left) hide)
     )
@@
       (effects (font (size 1.524 1.524)) (justify left) hide)
     )
-    (property "Footprint" "Package_TO_SOT_SMD:SOT-23" (id 2) (at 123.19 92.71 0)
-      (effects (font (size 1.524 1.524)) (justify left) hide)
-    )
+    (property "Footprint" "Package_TO_SOT_SMD:SOT-23_Handsoldering" (id 2) (at 123.19 92.71 0)
+      (effects (font (size 1.524 1.524)) (justify left) hide)
+    )

Commit message: schematics footer and export
Other:
- company: (none) -> Andrei Speridiao
- title: (none) -> E-TKT
Changed lines of the file:
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@@
 (kicad_sch (version 20211123) (generator eeschema)
   (paper "A4")
+  (title_block
+    (title "E-TKT")
+    (date "2022-07-21")
+    (rev "3")
+    (company "Andrei Speridiao")
+  )
   (junction (at 153.67 146.05) (diameter 0) (color 0 0 0 0)
   )
