File: _electronic/KiCad/charstepper.kicad_sch (KiCad schematic)
At the start: 8 parts

Commit message: revised IC packages, pins and footprints
Parts:
- C_NEMA1: footprint Capacitor_SMD:CP_Elec_6.3x5.9 -> Capacitor_SMD:CP_Elec_6.3x7.7
Changed lines of the file:
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@@
       (effects (font (size 1.27 1.27)) (justify left))
     )
-    (property "Footprint" "Capacitor_SMD:CP_Elec_6.3x5.9" (id 2) (at 183.8452 93.98 0)
+    (property "Footprint" "Capacitor_SMD:CP_Elec_6.3x7.7" (id 2) (at 183.8452 93.98 0)
       (effects (font (size 1.27 1.27)) hide)
     )

Commit message: schematics footer and export
Other:
- company: (none) -> Andrei Speridiao
- title: (none) -> E-TKT
Changed lines of the file:
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@@
 (kicad_sch (version 20211123) (generator eeschema)
   (paper "A4")
+  (title_block
+    (title "E-TKT")
+    (date "2022-07-21")
+    (rev "3")
+    (company "Andrei Speridiao")
+  )
   (junction (at 116.84 90.17) (diameter 0) (color 0 0 0 0)
   )
