File: _electronic/KiCad/connectors.kicad_sch (KiCad schematic)
At the start: 8 parts

Commit message: better buck layout and final revision
Parts:
- removed C_SERVO1: 22uF 12V 1mOhm, Capacitor_SMD:C_1210_3225Metric_Pad1.33x2.70mm_HandSolder, symbol Device:C
Changed lines of the file:
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@@
-    (stroke (width 0) (type default) (color 0 0 0 0))
-  )
-  (wire (pts (xy 137.16 82.55) (xy 137.16 83.82))
     (stroke (width 0) (type default) (color 0 0 0 0))
   )
@@
   )
   (wire (pts (xy 118.11 127) (xy 115.57 127))
-    (stroke (width 0) (type default) (color 0 0 0 0))
-  )
-  (wire (pts (xy 137.16 92.71) (xy 137.16 91.44))
     (stroke (width 0) (type default) (color 0 0 0 0))
   )
@@
     (effects (font (size 1.27 1.27)) (justify left))
   )
-  (hierarchical_label "6V IN" (shape input) (at 137.16 82.55 90)
-    (effects (font (size 1.27 1.27)) (justify left))
-  )
   (hierarchical_label "3V3 IN" (shape input) (at 138.43 125.73 90)
     (effects (font (size 1.27 1.27)) (justify left))
@@
     (pin "2")
     (pin "3")
-  )
-  (symbol (lib_id "Device:C") (at 137.16 87.63 0) (unit 1)
-    (in_bom yes) (on_board yes)
-    (property "Reference" "C_SERVO1" (id 0) (at 140.97 86.36 0)
-      (effects (font (size 1.27 1.27)) (justify left))
-    )
-    (property "Value" "22uF 12V 1mOhm" (id 1) (at 140.97 88.9 0)
-      (effects (font (size 1.27 1.27)) (justify left))
-    )
-    (property "Footprint" "Capacitor_SMD:C_1210_3225Metric_Pad1.33x2.70mm_HandSolder" (id 2) (at 138.1252 91.44 0)
-      (effects (font (size 1.27 1.27)) hide)
-    )
-    (property "Datasheet" "https://product.tdk.com/system/files/dam/doc/product/capacitor/ceramic/mlcc/catalog/mlcc_commercial_general_en.pdf?ref_disty=mouser" (id 3) (at 137.16 87.63 0)
-      (effects (font (size 1.27 1.27)) hide)
-    )
-    (property "#" "C3225X7R1E226M250AB" (id 4) (at 140.97 87.63 0)
-      (effects (font (size 1.27 1.27) italic) (justify left) hide)
-    )
-    (property "Description" "Decouple" (id 5) (at 137.16 87.63 0)
-      (effects (font (size 1.27 1.27)) hide)
-    )
-    (property "Group" "Servo" (id 6) (at 137.16 87.63 0)
-      (effects (font (size 1.27 1.27)) hide)
-    )
-    (property "Obs" "wes" (id 7) (at 137.16 87.63 0)
-      (effects (font (size 1.27 1.27)) hide)
-    )
-    (property "Mouser" "OK" (id 8) (at 137.16 87.63 0)
-      (effects (font (size 1.27 1.27)) hide)
-    )
-    (pin "1")
-    (pin "2")
   )
   (symbol (lib_id "Connector:Conn_01x03_Male") (at 110.49 86.36 0) (mirror x) (unit 1)
@@
     (pin "4")
   )
-  (symbol (lib_id "power:GNDREF") (at 137.16 92.71 0) (unit 1)
-    (in_bom yes) (on_board yes) (fields_autoplaced)
-    (property "Reference" "#PWR0129" (id 0) (at 137.16 99.06 0)
-      (effects (font (size 1.27 1.27)) hide)
-    )
-    (property "Value" "GNDREF" (id 1) (at 137.16 97.79 0)
-      (effects (font (size 1.27 1.27)) hide)
-    )
-    (property "Footprint" "" (id 2) (at 137.16 92.71 0)
-      (effects (font (size 1.27 1.27)) hide)
-    )
-    (property "Datasheet" "" (id 3) (at 137.16 92.71 0)
-      (effects (font (size 1.27 1.27)) hide)
-    )
-    (pin "1")
-  )
 )

Commit message: schematics footer and export
Other:
- company: (none) -> Andrei Speridiao
- title: (none) -> E-TKT
Changed lines of the file:
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@@
 (kicad_sch (version 20211123) (generator eeschema)
   (paper "A4")
+  (title_block
+    (title "E-TKT")
+    (date "2022-07-21")
+    (rev "3")
+    (company "Andrei Speridiao")
+  )
   (wire (pts (xy 138.43 129.54) (xy 138.43 125.73))
     (stroke (width 0) (type default) (color 0 0 0 0))
