File: _electronic/KiCad/feedstepper.kicad_sch (KiCad schematic)
At the start: 11 parts

Commit message: uln2003 soic narrow
Parts:
- U_STP1: footprint Package_SO:SOIC-16W_5.3x10.2mm_P1.27mm -> Package_SO:SOIC-16_3.9x9.9mm_P1.27mm; # ULN2003ADR2G -> ULN2003ADRE4
Changed lines of the file:
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@@
       (effects (font (size 1.27 1.27)) (justify left))
     )
-    (property "Footprint" "Package_SO:SOIC-16W_5.3x10.2mm_P1.27mm" (id 2) (at 124.46 127 0)
+    (property "Footprint" "Package_SO:SOIC-16_3.9x9.9mm_P1.27mm" (id 2) (at 124.46 127 0)
       (effects (font (size 1.27 1.27)) (justify left) hide)
     )
-    (property "Datasheet" "https://br.mouser.com/datasheet/2/308/1/ULN2003A_D-2320193.pdf" (id 3) (at 125.73 118.11 0)
+    (property "Datasheet" "https://www.ti.com/general/docs/suppproductinfo.tsp?distId=26&gotoUrl=https://www.ti.com/lit/gpn/uln2003a" (id 3) (at 125.73 118.11 0)
       (effects (font (size 1.27 1.27)) hide)
     )
-    (property "#" "ULN2003ADR2G" (id 5) (at 123.19 113.03 0)
+    (property "#" "ULN2003ADRE4" (id 5) (at 123.19 113.03 0)
       (effects (font (size 1.27 1.27)) hide)
     )

Commit message: schematics footer and export
Other:
- company: (none) -> Andrei Speridiao
- title: (none) -> E-TKT
Changed lines of the file:
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@@
 (kicad_sch (version 20211123) (generator eeschema)
   (paper "A4")
+  (title_block
+    (title "E-TKT")
+    (date "2022-07-21")
+    (rev "3")
+    (company "Andrei Speridiao")
+  )
   (junction (at 144.78 110.49) (diameter 0) (color 0 0 0 0)
   )
