File: _electronic/KiCad/levelshift.kicad_sch (KiCad schematic)
At the start: 10 parts

Commit message: revised IC packages, pins and footprints
Parts:
- Q_HALL1, Q_SERVO1: value BSS138 -> BSS138LT3G; footprint Package_TO_SOT_SMD:SOT-23 -> Package_TO_SOT_SMD:SOT-23_Handsoldering; # BSS138W-7-F -> BSS138LT3G
Changed lines of the file:
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@@
     (in_bom yes) (on_board yes)
     (property "Reference" "Q_HALL1" (id 0) (at 138.43 88.9 90))
-    (property "Value" "BSS138" (id 1) (at 138.43 87.63 90)
+    (property "Value" "BSS138LT3G" (id 1) (at 138.43 87.63 90)
       (effects (font (size 1.27 1.27)) hide)
     )
-    (property "Footprint" "Package_TO_SOT_SMD:SOT-23" (id 2) (at 140.335 90.17 0)
+    (property "Footprint" "Package_TO_SOT_SMD:SOT-23_Handsoldering" (id 2) (at 140.335 90.17 0)
       (effects (font (size 1.27 1.27) italic) (justify left) hide)
     )
-    (property "Datasheet" "https://www.diodes.com/assets/Datasheets/ds30206.pdf" (id 3) (at 138.43 95.25 0)
+    (property "Datasheet" "https://br.mouser.com/datasheet/2/308/1/BSS138LT1_D-2310401.pdf" (id 3) (at 138.43 95.25 0)
       (effects (font (size 1.27 1.27)) (justify left) hide)
     )
-    (property "#" "BSS138W-7-F" (id 4) (at 138.43 88.9 90)
+    (property "#" "BSS138LT3G" (id 4) (at 138.43 88.9 90)
       (effects (font (size 1.27 1.27) italic) hide)
     )
@@
     (in_bom yes) (on_board yes)
     (property "Reference" "Q_SERVO1" (id 0) (at 137.16 113.03 90))
-    (property "Value" "BSS138" (id 1) (at 137.16 111.76 90)
+    (property "Value" "BSS138LT3G" (id 1) (at 137.16 111.76 90)
       (effects (font (size 1.27 1.27)) hide)
     )
-    (property "Footprint" "Package_TO_SOT_SMD:SOT-23" (id 2) (at 139.065 114.3 0)
+    (property "Footprint" "Package_TO_SOT_SMD:SOT-23_Handsoldering" (id 2) (at 139.065 114.3 0)
       (effects (font (size 1.27 1.27) italic) (justify left) hide)
     )
-    (property "Datasheet" "https://www.diodes.com/assets/Datasheets/ds30206.pdf" (id 3) (at 137.16 119.38 0)
+    (property "Datasheet" "https://br.mouser.com/datasheet/2/308/1/BSS138LT1_D-2310401.pdf" (id 3) (at 137.16 119.38 0)
       (effects (font (size 1.27 1.27)) (justify left) hide)
     )
-    (property "#" "BSS138W-7-F" (id 4) (at 137.16 113.03 90)
+    (property "#" "BSS138LT3G" (id 4) (at 137.16 113.03 90)
       (effects (font (size 1.27 1.27) italic) hide)
     )

Commit message: schematics footer and export
Other:
- company: (none) -> Andrei Speridiao
- title: (none) -> E-TKT
Changed lines of the file:
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@@
 (kicad_sch (version 20211123) (generator eeschema)
   (paper "A4")
+  (title_block
+    (title "E-TKT")
+    (date "2022-07-21")
+    (rev "3")
+    (company "Andrei Speridiao")
+  )
   (junction (at 144.78 116.84) (diameter 0) (color 0 0 0 0)
   )
