File: _electronic/KiCad/testpads.kicad_sch (KiCad schematic)
At the start: 11 parts

Commit message: added buzzer
Parts:
- removed TP_GND2: TestPoint, TestPoint:TestPoint_Pad_D1.0mm, symbol Connector:TestPoint
Changed lines of the file:
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@@
 (kicad_sch (version 20211123) (generator eeschema)
   (paper "A4")
-  (junction (at 187.96 109.22) (diameter 0) (color 0 0 0 0)
-  )
   (wire (pts (xy 186.69 109.22) (xy 187.96 109.22))
     (stroke (width 0) (type default) (color 0 0 0 0))
@@
     (stroke (width 0) (type default) (color 0 0 0 0))
   )
-  (wire (pts (xy 186.69 95.25) (xy 187.96 95.25))
-    (stroke (width 0) (type default) (color 0 0 0 0))
-  )
   (wire (pts (xy 153.67 95.25) (xy 152.4 95.25))
     (stroke (width 0) (type default) (color 0 0 0 0))
   )
   (wire (pts (xy 153.67 107.95) (xy 153.67 109.22))
-    (stroke (width 0) (type default) (color 0 0 0 0))
-  )
-  (wire (pts (xy 187.96 95.25) (xy 187.96 109.22))
     (stroke (width 0) (type default) (color 0 0 0 0))
   )
@@
       (effects (font (size 1.27 1.27)) hide)
     )
-    (pin "1")
-  )
-  (symbol (lib_id "Connector:TestPoint") (at 186.69 95.25 90) (unit 1)
-    (in_bom yes) (on_board yes)
-    (property "Reference" "TP_GND2" (id 0) (at 181.61 95.25 90)
-      (effects (font (size 1.27 1.27)) (justify left))
-    )
-    (property "Value" "TestPoint" (id 1) (at 181.61 95.25 90)
-      (effects (font (size 1.27 1.27)) (justify left) hide)
-    )
-    (property "Footprint" "TestPoint:TestPoint_Pad_D1.0mm" (id 2) (at 186.69 90.17 0)
-      (effects (font (size 1.27 1.27)) hide)
-    )
-    (property "Datasheet" "xxx" (id 3) (at 186.69 90.17 0)
-      (effects (font (size 1.27 1.27)) hide)
-    )
-    (property "#" "xxx" (id 5) (at 186.69 95.25 0)
-      (effects (font (size 1.27 1.27)) hide)
-    )
-    (property "Description" "Testing point" (id 6) (at 186.69 95.25 0)
-      (effects (font (size 1.27 1.27)) hide)
-    )
-    (property "Group" "Pads" (id 4) (at 186.69 95.25 0)
-      (effects (font (size 1.27 1.27)) hide)
-    )
-    (property "Mouser" "OK" (id 7) (at 186.69 95.25 0)
-      (effects (font (size 1.27 1.27)) hide)
-    )

Commit message: schematics footer and export
Other:
- company: (none) -> Andrei Speridiao
- title: (none) -> E-TKT
Changed lines of the file:
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@@
 (kicad_sch (version 20211123) (generator eeschema)
   (paper "A4")
+  (title_block
+    (title "E-TKT")
+    (date "2022-07-21")
+    (rev "3")
+    (company "Andrei Speridiao")
+  )
   (wire (pts (xy 186.69 109.22) (xy 187.96 109.22))
     (stroke (width 0) (type default) (color 0 0 0 0))
