File: _electronic/KiCad/usb.kicad_sch (KiCad schematic)
At the start: 8 parts

Commit message: schematics footer and export
Other:
- company: (none) -> Andrei Speridiao
- title: (none) -> E-TKT
Changed lines of the file:
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@@
 (kicad_sch (version 20211123) (generator eeschema)
   (paper "A4")
+  (title_block
+    (title "E-TKT")
+    (date "2022-07-21")
+    (rev "3")
+    (company "Andrei Speridiao")
+  )
   (junction (at 143.51 113.03) (diameter 0) (color 0 0 0 0)
   )
