File: _electronic/extflashing.kicad_sch (KiCad schematic)
At the start: 1 part

Commit message: organized electronics folder
Parts:
- J_EXT1: # (none) -> xxx; Mouser (none) -> OK
Changed lines of the file:
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@@
+      (effects (font (size 1.27 1.27)) hide)
+    )
+    (property "#" "xxx" (id 4) (at 135.89 113.03 0)
+      (effects (font (size 1.27 1.27)) hide)
+    )
+    (property "Mouser" "OK" (id 5) (at 135.89 113.03 0)
       (effects (font (size 1.27 1.27)) hide)
     )
