File: _electronic/e-tkt.kicad_pcb (KiCad board)
At the start: 4 copper layers, 99.6 x 76.2 mm, 108 parts

Commit message: v1 pcb
Parts:
- removed the REF** at (178.3, -198.9)
- added G***: LOGO, LOGO, F.Cu at (147.1, -222.8)
- added G***: LOGO, LOGO, B.Cu at (209.6, -222.2)
- added REF**: OSHW-Symbol_6.7x6mm_SilkScreen, andrei custom:opengear_small, F.Cu at (155.2, -205.0)
- moved C_MCU2 2.03 mm to (163.1, -217.4)
- moved C_MCU1 2.03 mm to (165.1, -217.4)
- moved C_STP1 1.37 mm to (150.6, -177.0)
- moved J_NEMA1 1.27 mm to (208.5, -181.1)
- moved LS1 0.72 mm to (143.3, -200.7), turned to -90 degrees
- moved G*** 0.51 mm to (178.3, -191.8)
- moved D_USB1 0.25 mm to (141.2, -178.3)
- moved D_POW2 0.25 mm to (141.2, -174.2)
- moved G*** 0.25 mm to (178.3, -189.0)
- moved R_POW6 0.25 mm to (141.2, -176.3)
- moved R_USB1 0.25 mm to (145.0, -181.6)
- moved R_USB2 0.25 mm to (141.2, -181.6)
- moved G*** 0.24 mm to (178.3, -189.2)
- moved C_NEMA2 0.09 mm to (183.8, -169.4)
- renumbered C_RST1 to C_DFU1, R_RST1 to R_DFU1, SW_RST1 to SW_DFU1
Connections:
- net IO0 RESET renamed IO0 DFU
- LS1 pad 1: /MCU/IO27 BUZZER OUT -> /MCU/IO26 BUZZER OUT
- U_MCU1 pad 11: unconnected-(U_MCU1-Pad11) -> /MCU/IO26 BUZZER OUT
- U_MCU1 pad 12: /MCU/IO27 BUZZER OUT -> unconnected-(U_MCU1-Pad12)
Routing:
- net /MCU/IO26 BUZZER OUT: track 0.00 -> 33.3 mm, vias 0 -> 2
- net /MCU/IO27 BUZZER OUT: track 27.5 -> 0.00 mm, vias 2 -> 0
- net EN: track 66.5 -> 69.7 mm
- net IO17 LED PRESS: track 53.4 -> 51.8 mm
- net +3.3V: track 232.2 -> 231.2 mm
- net IO21 OLED SDA: track 38.6 -> 37.8 mm
- net +12V: track 250.3 -> 251.2 mm, vias 29 -> 33
- net +6V: track 107.3 -> 108.1 mm
- net Net-(A_NEMA1-Pad3): track 40.6 -> 41.4 mm
- net Net-(A_NEMA1-Pad4): track 40.7 -> 41.3 mm
- net IO22 OLED SCL: track 33.1 -> 32.5 mm
- net IO14 SERVO: track 77.0 -> 76.4 mm
- net Net-(A_NEMA1-Pad5): track 40.8 -> 41.3 mm
- net Net-(A_NEMA1-Pad6): track 40.3 -> 40.9 mm
- net GNDREF: vias 360 -> 351

Commit message: fn label on silkscreen
Other:
- board text added: "*"
