File: _electronic/e-tkt.kicad_pcb (KiCad board)
At the start: 4 copper layers, 99.6 x 76.2 mm, 110 parts

Commit message: fixed hall header on pcb
Parts:
- J_HALL1: footprint Connector_PinSocket_2.54mm:PinSocket_1x03_P2.54mm_Vertical -> Connector_PinHeader_2.54mm:PinHeader_1x03_P2.54mm_Vertical
Changed lines of the file:
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@@
     )
   )
-  (footprint "Connector_PinSocket_2.54mm:PinSocket_1x03_P2.54mm_Vertical" (layer "B.Cu")
+  (footprint "Connector_PinHeader_2.54mm:PinHeader_1x03_P2.54mm_Vertical" (layer "B.Cu")
     (at 214.884 -187.452 90)
-    (descr "Through hole straight socket strip, 1x03, 2.54mm pitch, single row (from Kicad 4.0.7), script generated")
-    (tags "Through hole socket strip THT 1x03 2.54mm single row")
+    (descr "Through hole straight pin header, 1x03, 2.54mm pitch, single row")
+    (tags "Through hole pin header THT 1x03 2.54mm single row")
     (property "#" "M20-7820346")
     (property "Description" "Header")
@@
     (property "Sheetname" "Connectors")
     (attr through_hole)
-    (fp_text reference "J_HALL1" (at 0 2.77 270) (layer "B.SilkS") hide
+    (fp_text reference "J_HALL1" (at 0 2.33 270) (layer "B.SilkS") hide
       (effects (font (size 1 1) (thickness 0.15)) (justify mirror))
     )
-    (fp_text value "Conn_01x03_Female" (at 0 -7.85 270) (layer "B.Fab")
+    (fp_text value "Conn_01x03_Female" (at 0 -7.41 270) (layer "B.Fab")
       (effects (font (size 1 1) (thickness 0.15)) (justify mirror))
     )
@@
       (effects (font (size 1 1) (thickness 0.15)) (justify mirror))
     )
+    (fp_line (start -1.33 0) (end -1.33 1.33) (layer "B.SilkS") (width 0.12))
     (fp_line (start -1.33 -1.27) (end 1.33 -1.27) (layer "B.SilkS") (width 0.12))
-    (fp_line (start 1.33 1.33) (end 1.33 0) (layer "B.SilkS") (width 0.12))
+    (fp_line (start -1.33 -1.27) (end -1.33 -6.41) (layer "B.SilkS") (width 0.12))
+    (fp_line (start -1.33 1.33) (end 0 1.33) (layer "B.SilkS") (width 0.12))
     (fp_line (start -1.33 -6.41) (end 1.33 -6.41) (layer "B.SilkS") (width 0.12))
-    (fp_line (start 0 1.33) (end 1.33 1.33) (layer "B.SilkS") (width 0.12))
-    (fp_line (start -1.33 -1.27) (end -1.33 -6.41) (layer "B.SilkS") (width 0.12))
     (fp_line (start 1.33 -1.27) (end 1.33 -6.41) (layer "B.SilkS") (width 0.12))
-    (fp_line (start 1.75 -6.85) (end -1.8 -6.85) (layer "B.CrtYd") (width 0.05))
-    (fp_line (start -1.8 1.8) (end 1.75 1.8) (layer "B.CrtYd") (width 0.05))
-    (fp_line (start -1.8 -6.85) (end -1.8 1.8) (layer "B.CrtYd") (width 0.05))
-    (fp_line (start 1.75 1.8) (end 1.75 -6.85) (layer "B.CrtYd") (width 0.05))
-    (fp_line (start -1.27 1.27) (end 0.635 1.27) (layer "B.Fab") (width 0.1))
-    (fp_line (start 1.27 0.635) (end 1.27 -6.35) (layer "B.Fab") (width 0.1))
+    (fp_line (start -1.8 -6.85) (end 1.8 -6.85) (layer "B.CrtYd") (width 0.05))
+    (fp_line (start 1.8 1.8) (end -1.8 1.8) (layer "B.CrtYd") (width 0.05))
+    (fp_line (start -1.8 1.8) (end -1.8 -6.85) (layer "B.CrtYd") (width 0.05))
+    (fp_line (start 1.8 -6.85) (end 1.8 1.8) (layer "B.CrtYd") (width 0.05))
+    (fp_line (start 1.27 1.27) (end 1.27 -6.35) (layer "B.Fab") (width 0.1))
     (fp_line (start 1.27 -6.35) (end -1.27 -6.35) (layer "B.Fab") (width 0.1))
-    (fp_line (start -1.27 -6.35) (end -1.27 1.27) (layer "B.Fab") (width 0.1))
-    (fp_line (start 0.635 1.27) (end 1.27 0.635) (layer "B.Fab") (width 0.1))
+    (fp_line (start -1.27 0.635) (end -0.635 1.27) (layer "B.Fab") (width 0.1))
+    (fp_line (start -0.635 1.27) (end 1.27 1.27) (layer "B.Fab") (width 0.1))
+    (fp_line (start -1.27 -6.35) (end -1.27 0.635) (layer "B.Fab") (width 0.1))
     (pad "1" thru_hole rect (at 0 0 90) (size 1.7 1.7) (drill 1) (layers *.Cu *.Mask)
       (net 2 "GNDREF") (pinfunction "Pin_1") (pintype "passive"))
