File: _electronic/testpads.kicad_sch (KiCad schematic)
At the start: 10 parts

Commit message: v1 pcb
Parts:
- removed TP_12v1, TP_3.3v1, TP_5v1, TP_6v1, TP_GND3: TestPoint, TestPoint:TestPoint_Pad_D1.0mm, symbol Connector:TestPoint
Changed lines of the file:
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@@
     (effects (font (size 1.27 1.27)) (justify left))
-  )
-  (symbol (lib_id "Connector:TestPoint") (at 168.91 95.25 90) (unit 1)
-    (in_bom yes) (on_board yes)
-    (property "Reference" "TP_6v1" (id 0) (at 163.83 95.25 90)
-      (effects (font (size 1.27 1.27)) (justify left))
-    )
-    (property "Value" "TestPoint" (id 1) (at 163.83 95.25 90)
-      (effects (font (size 1.27 1.27)) (justify left) hide)
-    )
-    (property "Footprint" "TestPoint:TestPoint_Pad_D1.0mm" (id 2) (at 168.91 90.17 0)
-      (effects (font (size 1.27 1.27)) hide)
-    )
-    (property "Datasheet" "xxx" (id 3) (at 168.91 90.17 0)
-      (effects (font (size 1.27 1.27)) hide)
-    )
-    (property "#" "xxx" (id 5) (at 168.91 95.25 0)
-      (effects (font (size 1.27 1.27)) hide)
-    )
-    (property "Description" "Testing point" (id 6) (at 168.91 95.25 0)
-      (effects (font (size 1.27 1.27)) hide)
-    )
-    (property "Group" "Pads" (id 4) (at 168.91 95.25 0)
-      (effects (font (size 1.27 1.27)) hide)
-    )
-    (property "Mouser" "OK" (id 7) (at 168.91 95.25 0)
-      (effects (font (size 1.27 1.27)) hide)
-    )
-    (pin "1")
   )
   (symbol (lib_id "power:GNDREF") (at 130.81 93.98 0) (unit 1)
@@
     (pin "1")
   )
-  (symbol (lib_id "Connector:TestPoint") (at 152.4 109.22 90) (unit 1)
-    (in_bom yes) (on_board yes)
-    (property "Reference" "TP_5v1" (id 0) (at 147.32 109.22 90)
-      (effects (font (size 1.27 1.27)) (justify left))
-    )
-    (property "Value" "TestPoint" (id 1) (at 147.32 109.22 90)
-      (effects (font (size 1.27 1.27)) (justify left) hide)
-    )
-    (property "Footprint" "TestPoint:TestPoint_Pad_D1.0mm" (id 2) (at 152.4 104.14 0)
-      (effects (font (size 1.27 1.27)) hide)
-    )
-    (property "Datasheet" "xxx" (id 3) (at 152.4 104.14 0)
-      (effects (font (size 1.27 1.27)) hide)
-    )
-    (property "#" "xxx" (id 5) (at 152.4 109.22 0)
-      (effects (font (size 1.27 1.27)) hide)
-    )
-    (property "Description" "Testing point" (id 6) (at 152.4 109.22 0)
-      (effects (font (size 1.27 1.27)) hide)
-    )
-    (property "Group" "Pads" (id 4) (at 152.4 109.22 0)
-      (effects (font (size 1.27 1.27)) hide)
-    )
-    (property "Mouser" "OK" (id 7) (at 152.4 109.22 0)
-      (effects (font (size 1.27 1.27)) hide)
-    )
-    (pin "1")
-  )
-  (symbol (lib_id "Connector:TestPoint") (at 168.91 109.22 90) (unit 1)
-    (in_bom yes) (on_board yes)
-    (property "Reference" "TP_12v1" (id 0) (at 163.83 109.22 90)
-      (effects (font (size 1.27 1.27)) (justify left))
-    )
-    (property "Value" "TestPoint" (id 1) (at 163.83 109.22 90)
-      (effects (font (size 1.27 1.27)) (justify left) hide)
-    )
-    (property "Footprint" "TestPoint:TestPoint_Pad_D1.0mm" (id 2) (at 168.91 104.14 0)
-      (effects (font (size 1.27 1.27)) hide)
-    )
-    (property "Datasheet" "xxx" (id 3) (at 168.91 104.14 0)
-      (effects (font (size 1.27 1.27)) hide)
-    )
-    (property "Group" "Pads" (id 4) (at 168.91 109.22 0)
-      (effects (font (size 1.27 1.27)) hide)
-    )
-    (property "#" "xxx" (id 5) (at 168.91 109.22 0)
-      (effects (font (size 1.27 1.27)) hide)
-    )
-    (property "Description" "Testing point" (id 6) (at 168.91 109.22 0)
-      (effects (font (size 1.27 1.27)) hide)
-    )
-    (property "Mouser" "OK" (id 7) (at 168.91 109.22 0)
-      (effects (font (size 1.27 1.27)) hide)
-    )
-    (pin "1")
-  )
-  (symbol (lib_id "Connector:TestPoint") (at 152.4 95.25 90) (unit 1)
-    (in_bom yes) (on_board yes)
-    (property "Reference" "TP_3.3v1" (id 0) (at 147.32 95.25 90)
-      (effects (font (size 1.27 1.27)) (justify left))
-    )
-    (property "Value" "TestPoint" (id 1) (at 147.32 95.25 90)
-      (effects (font (size 1.27 1.27)) (justify left) hide)
-    )
-    (property "Footprint" "TestPoint:TestPoint_Pad_D1.0mm" (id 2) (at 152.4 90.17 0)
-      (effects (font (size 1.27 1.27)) hide)
-    )
-    (property "Datasheet" "xxx" (id 3) (at 152.4 90.17 0)
-      (effects (font (size 1.27 1.27)) hide)
-    )
-    (property "#" "xxx" (id 6) (at 152.4 95.25 0)
-      (effects (font (size 1.27 1.27)) hide)
-    )
-    (property "Group" "Pads" (id 4) (at 152.4 95.25 0)
-      (effects (font (size 1.27 1.27)) hide)
-    )
-    (property "Description" "Testing point" (id 5) (at 152.4 95.25 0)
-      (effects (font (size 1.27 1.27)) hide)
-    )
-    (property "Mouser" "OK" (id 7) (at 152.4 95.25 0)
-      (effects (font (size 1.27 1.27)) hide)
-    )
-    (pin "1")
-  )
   (symbol (lib_id "Mechanical:MountingHole_Pad") (at 128.27 107.95 90) (unit 1)
     (in_bom yes) (on_board yes)
@@
       (effects (font (size 1.27 1.27)) hide)
     )
-    (pin "1")
-  )
-  (symbol (lib_id "Connector:TestPoint") (at 186.69 109.22 90) (unit 1)
-    (in_bom yes) (on_board yes)
-    (property "Reference" "TP_GND3" (id 0) (at 181.61 109.22 90)
-      (effects (font (size 1.27 1.27)) (justify left))
-    )
-    (property "Value" "TestPoint" (id 1) (at 181.61 109.22 90)
-      (effects (font (size 1.27 1.27)) (justify left) hide)
-    )
-    (property "Footprint" "TestPoint:TestPoint_Pad_D1.0mm" (id 2) (at 186.69 104.14 0)
-      (effects (font (size 1.27 1.27)) hide)
-    )
-    (property "Datasheet" "xxx" (id 3) (at 186.69 104.14 0)
-      (effects (font (size 1.27 1.27)) hide)
-    )
-    (property "#" "xxx" (id 5) (at 186.69 109.22 0)
-      (effects (font (size 1.27 1.27)) hide)
-    )
-    (property "Description" "Testing point" (id 6) (at 186.69 109.22 0)
-      (effects (font (size 1.27 1.27)) hide)
-    )
-    (property "Group" "Pads" (id 4) (at 186.69 109.22 0)
-      (effects (font (size 1.27 1.27)) hide)
-    )
-    (property "Mouser" "OK" (id 7) (at 186.69 109.22 0)
-      (effects (font (size 1.27 1.27)) hide)
-    )

Commit message: led resistor revision, b.o.m. and pcb anotation
Other:
- moved on the sheet: H1, H2, H3, H4, H6
