File: _electronic/boot.kicad_sch (KiCad schematic)
At the start: 10 parts

Commit message: organized electronics folder
Parts:
- C_ENA1, C_RST1: value 0.1uF 10V -> 0.1uF 50V; # CGA3E2X7R1H104K080AA -> C1608X7R1H104K080AA
Changed lines of the file:
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@@
       (effects (font (size 1.27 1.27)) (justify right))
     )
-    (property "Value" "0.1uF 10V" (id 1) (at 193.04 88.9 0)
+    (property "Value" "0.1uF 50V" (id 1) (at 193.04 88.9 0)
       (effects (font (size 1.27 1.27)) (justify right))
     )
@@
       (effects (font (size 1.27 1.27)) hide)
     )
-    (property "#" "CGA3E2X7R1H104K080AA" (id 4) (at 204.47 87.63 0)
+    (property "#" "C1608X7R1H104K080AA" (id 4) (at 204.47 87.63 0)
       (effects (font (size 1.27 1.27) italic) hide)
     )
@@
       (effects (font (size 1.27 1.27)) (justify right))
     )
-    (property "Value" "0.1uF 10V" (id 1) (at 193.04 138.43 0)
+    (property "Value" "0.1uF 50V" (id 1) (at 193.04 138.43 0)
       (effects (font (size 1.27 1.27)) (justify right))
     )
@@
       (effects (font (size 1.27 1.27)) hide)
     )
-    (property "#" "CGA3E2X7R1H104K080AA" (id 4) (at 205.74 137.16 0)
+    (property "#" "C1608X7R1H104K080AA" (id 4) (at 205.74 137.16 0)
       (effects (font (size 1.27 1.27) italic) hide)
     )

Commit message: v1 pcb
Parts:
- renumbered C_RST1 to C_DFU1, R_RST1 to R_DFU1, SW_RST1 to SW_DFU1
Connections:
- net RESET OUT renamed DFU OUT
Changed lines of the file:
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@@
     (effects (font (size 1.27 1.27)) (justify left))
   )
-  (hierarchical_label "RESET OUT" (shape input) (at 127 123.19 0)
+  (hierarchical_label "DFU OUT" (shape input) (at 127 123.19 0)
     (effects (font (size 1.27 1.27)) (justify left))
   )
@@
     (effects (font (size 1.27 1.27)) (justify right))
   )
-  (hierarchical_label "RESET OUT" (shape input) (at 193.04 130.81 0)
+  (hierarchical_label "DFU OUT" (shape input) (at 193.04 130.81 0)
     (effects (font (size 1.27 1.27)) (justify left))
   )
@@
   (symbol (lib_id "Device:R") (at 189.23 123.19 0) (unit 1)
     (in_bom yes) (on_board yes)
-    (property "Reference" "R_RST1" (id 0) (at 191.77 121.92 0)
+    (property "Reference" "R_DFU1" (id 0) (at 191.77 121.92 0)
       (effects (font (size 1.27 1.27)) (justify left))
     )
@@
   (symbol (lib_id "Device:C") (at 189.23 137.16 180) (unit 1)
     (in_bom yes) (on_board yes)
-    (property "Reference" "C_RST1" (id 0) (at 193.04 135.89 0)
+    (property "Reference" "C_DFU1" (id 0) (at 193.04 135.89 0)
       (effects (font (size 1.27 1.27)) (justify right))
     )
@@
   (symbol (lib_id "2022-07-12_23-59-33:B3FS-1000") (at 162.56 152.4 90) (unit 1)
     (in_bom yes) (on_board yes)
-    (property "Reference" "SW_RST1" (id 0) (at 167.64 121.92 90)
+    (property "Reference" "SW_DFU1" (id 0) (at 167.64 121.92 90)
       (effects (font (size 1.524 1.524)) (justify right))
     )

Commit message: led resistor revision, b.o.m. and pcb anotation
Parts:
- R_AUTO1, R_AUTO2, R_DFU1, R_ENA1: value 10K (5%) -> 10K; # CHP0603AFX-1002ELF -> ERJ-3EKF1002V
Changed lines of the file:
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@@
     (in_bom yes) (on_board yes)
     (property "Reference" "R_AUTO1" (id 0) (at 106.68 95.25 90))
-    (property "Value" "10K (5%)" (id 1) (at 106.68 100.33 90))
+    (property "Value" "10K" (id 1) (at 106.68 97.79 90))
     (property "Footprint" "Resistor_SMD:R_0603_1608Metric_Pad0.98x0.95mm_HandSolder" (id 2) (at 106.68 99.568 90)
       (effects (font (size 1.27 1.27)) hide)
@@
       (effects (font (size 1.27 1.27)) hide)
     )
-    (property "#" "CHP0603AFX-1002ELF" (id 4) (at 106.68 91.44 90)
+    (property "#" "ERJ-3EKF1002V" (id 4) (at 106.68 91.44 90)
       (effects (font (size 1.27 1.27) italic) hide)
     )
@@
       (effects (font (size 1.27 1.27)) (justify left))
     )
-    (property "Value" "10K (5%)" (id 1) (at 191.77 124.46 0)
-      (effects (font (size 1.27 1.27)) (justify left))
-    )
+    (property "Value" "10K" (id 1) (at 189.23 123.19 90))
     (property "Footprint" "Resistor_SMD:R_0603_1608Metric_Pad0.98x0.95mm_HandSolder" (id 2) (at 187.452 123.19 90)
       (effects (font (size 1.27 1.27)) hide)
@@
       (effects (font (size 1.27 1.27)) hide)
     )
-    (property "#" "CHP0603AFX-1002ELF" (id 4) (at 191.77 123.19 0)
+    (property "#" "ERJ-3EKF1002V" (id 4) (at 191.77 123.19 0)
       (effects (font (size 1.27 1.27) italic) (justify left) hide)
     )
@@
     (in_bom yes) (on_board yes)
     (property "Reference" "R_AUTO2" (id 0) (at 106.68 113.03 90))
-    (property "Value" "10K (5%)" (id 1) (at 106.68 118.11 90))
+    (property "Value" "10K" (id 1) (at 106.68 115.57 90))
     (property "Footprint" "Resistor_SMD:R_0603_1608Metric_Pad0.98x0.95mm_HandSolder" (id 2) (at 106.68 117.348 90)
       (effects (font (size 1.27 1.27)) hide)
@@
       (effects (font (size 1.27 1.27)) hide)
     )
-    (property "#" "CHP0603AFX-1002ELF" (id 4) (at 106.68 115.57 90)
+    (property "#" "ERJ-3EKF1002V" (id 4) (at 106.68 115.57 90)
       (effects (font (size 1.27 1.27)) hide)
     )
@@
       (effects (font (size 1.27 1.27)) (justify right))
     )
-    (property "Value" "10K (5%)" (id 1) (at 191.77 74.93 0)
-      (effects (font (size 1.27 1.27)) (justify right))
-    )
+    (property "Value" "10K" (id 1) (at 189.23 73.66 90))
     (property "Footprint" "Resistor_SMD:R_0603_1608Metric_Pad0.98x0.95mm_HandSolder" (id 2) (at 191.008 73.66 90)
       (effects (font (size 1.27 1.27)) hide)
@@
       (effects (font (size 1.27 1.27)) hide)
     )
-    (property "#" "CHP0603AFX-1002ELF" (id 4) (at 191.77 73.6601 0)
+    (property "#" "ERJ-3EKF1002V" (id 4) (at 191.77 73.6601 0)
       (effects (font (size 1.27 1.27) italic) (justify right) hide)
     )

Commit message: schematics and pcb cleanup
Other:
- title: E-TKT -> E-TKT v1.0
Changed lines of the file:
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@@
   (paper "A4")
   (title_block
-    (title "E-TKT")
-    (date "2022-07-21")
-    (rev "3")
+    (title "E-TKT v1.0")
+    (date "2022-09-29")
+    (rev "4")
     (company "Andrei Speridiao")
   )
