File: _electronic/power3v3.kicad_sch (KiCad schematic)
At the start: 3 parts

Commit message: led resistor revision, b.o.m. and pcb anotation
Parts:
- C_POW1: value 10uF 12V 5mOhm -> 10uF 12V; # C1608X5R1E106M080AC -> GRM188Z71A106KA73D
- C_POW2: value 22uF 12V 1mOhm -> 10uF 12V; # CL10A226MO7JZNC -> GRM188Z71A106KA73D
Changed lines of the file:
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@@
       (effects (font (size 1.27 1.27)) (justify right))
     )
-    (property "Value" "10uF 12V 5mOhm" (id 1) (at 123.19 107.95 0)
+    (property "Value" "10uF 12V" (id 1) (at 123.19 107.95 0)
       (effects (font (size 1.27 1.27)) (justify right))
     )
@@
       (effects (font (size 1.27 1.27)) hide)
     )
-    (property "#" "C1608X5R1E106M080AC" (id 4) (at 130.81 105.41 0)
+    (property "#" "GRM188Z71A106KA73D" (id 4) (at 130.81 105.41 0)
       (effects (font (size 1.27 1.27) italic) (justify left) hide)
     )
@@
       (effects (font (size 1.27 1.27)) (justify left))
     )
-    (property "Value" "22uF 12V 1mOhm" (id 1) (at 179.07 107.95 0)
+    (property "Value" "10uF 12V" (id 1) (at 179.07 107.95 0)
       (effects (font (size 1.27 1.27)) (justify left))
     )
@@
       (effects (font (size 1.27 1.27)) hide)
     )
-    (property "#" "CL10A226MO7JZNC" (id 7) (at 175.26 106.68 0)
+    (property "#" "GRM188Z71A106KA73D" (id 7) (at 175.26 106.68 0)
       (effects (font (size 1.27 1.27)) hide)
     )

Commit message: schematics and pcb cleanup
Other:
- title: E-TKT -> E-TKT v1.0
Changed lines of the file:
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@@
   (paper "A4")
   (title_block
-    (title "E-TKT")
-    (date "2022-07-21")
-    (rev "3")
+    (title "E-TKT v1.0")
+    (date "2022-09-29")
+    (rev "4")
     (company "Andrei Speridiao")
   )
