File: _electronic/wifireset.kicad_sch (KiCad schematic)
At the start: 3 parts

Commit message: organized electronics folder
Parts:
- C_WIFI1: value 0.1uF 10V -> 0.1uF 50V; # CGA3E2X7R1H104K080AA -> C1608X7R1H104K080AA
Changed lines of the file:
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@@
       (effects (font (size 1.27 1.27)) (justify right))
     )
-    (property "Value" "0.1uF 10V" (id 1) (at 163.83 107.95 0)
+    (property "Value" "0.1uF 50V" (id 1) (at 163.83 107.95 0)
       (effects (font (size 1.27 1.27)) (justify right))
     )
@@
       (effects (font (size 1.27 1.27)) hide)
     )
-    (property "#" "CGA3E2X7R1H104K080AA" (id 4) (at 176.53 106.68 0)
+    (property "#" "C1608X7R1H104K080AA" (id 4) (at 176.53 106.68 0)
       (effects (font (size 1.27 1.27) italic) hide)
     )

Commit message: led resistor revision, b.o.m. and pcb anotation
Parts:
- R_WIFI1: value 10K(5%) -> 10K; # CHP0603AFX-1002ELF -> ERJ-3EKF1002V
Changed lines of the file:
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@@
       (effects (font (size 1.27 1.27)) (justify right))
     )
-    (property "Value" "10K(5%)" (id 1) (at 162.56 93.98 0)
-      (effects (font (size 1.27 1.27)) (justify right))
-    )
+    (property "Value" "10K" (id 1) (at 160.02 92.71 90))
     (property "Footprint" "Resistor_SMD:R_0603_1608Metric_Pad0.98x0.95mm_HandSolder" (id 2) (at 161.798 92.71 90)
       (effects (font (size 1.27 1.27)) hide)
@@
       (effects (font (size 1.27 1.27)) hide)
     )
-    (property "#" "CHP0603AFX-1002ELF" (id 4) (at 162.56 92.71 0)
+    (property "#" "ERJ-3EKF1002V" (id 4) (at 162.56 92.71 0)
       (effects (font (size 1.27 1.27) italic) (justify right) hide)
     )

Commit message: schematics and pcb cleanup
Other:
- title: E-TKT -> E-TKT v1.0
Changed lines of the file:
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@@
   (paper "A4")
   (title_block
-    (title "E-TKT")
-    (date "2022-07-21")
-    (rev "3")
+    (title "E-TKT v1.0")
+    (date "2022-09-29")
+    (rev "4")
     (company "Andrei Speridiao")
   )
